File: i2cgpio.kicad_sch (KiCad schematic)
At the start: 4 parts

Commit message: respin
Parts:
- gave numbers to parts that had none: 4
Changed lines of the file:
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@@
   (symbol (lib_id "Device:C_Small") (at 45.72 53.34 0) (unit 1)
     (in_bom yes) (on_board yes)
-    (property "Reference" "C?" (id 0) (at 47.625 52.07 0)
+    (property "Reference" "C3" (id 0) (at 47.625 52.07 0)
       (effects (font (size 1.27 1.27)) (justify left))
     )
@@
   (symbol (lib_id "power:GND") (at 96.52 93.98 0) (unit 1)
     (in_bom yes) (on_board yes) (fields_autoplaced)
-    (property "Reference" "#PWR?" (id 0) (at 96.52 100.33 0)
+    (property "Reference" "#PWR05" (id 0) (at 96.52 100.33 0)
       (effects (font (size 1.27 1.27)) hide)
     )
@@
   (symbol (lib_id "Interface_I2C_NXP:PCA9671BS,118") (at 96.52 45.72 0) (unit 1)
     (in_bom yes) (on_board yes)
-    (property "Reference" "U?" (id 0) (at 106.68 41.91 0)
+    (property "Reference" "U2" (id 0) (at 106.68 41.91 0)
       (effects (font (size 1.524 1.524)))
     )
@@
   (symbol (lib_id "power:GND") (at 55.88 93.98 0) (unit 1)
     (in_bom yes) (on_board yes) (fields_autoplaced)
-    (property "Reference" "#PWR?" (id 0) (at 55.88 100.33 0)
+    (property "Reference" "#PWR04" (id 0) (at 55.88 100.33 0)
       (effects (font (size 1.27 1.27)) hide)
     )
@@
   (symbol (lib_id "Device:R_Small") (at 66.04 66.04 180) (unit 1)
     (in_bom yes) (on_board yes)
-    (property "Reference" "R?" (id 0) (at 69.85 64.77 0))
+    (property "Reference" "R1" (id 0) (at 69.85 64.77 0))
     (property "Value" "5.1k" (id 1) (at 69.85 67.31 0))
     (property "Footprint" "Resistor_SMD:R_0402_1005Metric" (id 2) (at 66.04 66.04 0)
@@
   (symbol (lib_id "Device:C_Small") (at 55.88 53.34 0) (unit 1)
     (in_bom yes) (on_board yes)
-    (property "Reference" "C?" (id 0) (at 57.785 52.07 0)
+    (property "Reference" "C4" (id 0) (at 57.785 52.07 0)
       (effects (font (size 1.27 1.27)) (justify left))
     )
