File: i2cgpio.kicad_sch (KiCad schematic)
At the start: 4 parts, among them U2 PCA9671BS,118

Commit message: work on control logic
Parts:
- renumbered R1 to R3
Changed lines of the file:
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@@
   (symbol (lib_id "Device:R_Small") (at 66.04 66.04 180) (unit 1)
     (in_bom yes) (on_board yes)
-    (property "Reference" "R1" (id 0) (at 69.85 64.77 0))
+    (property "Reference" "R3" (id 0) (at 69.85 64.77 0))
     (property "Value" "5.1k" (id 1) (at 69.85 67.31 0))
     (property "Footprint" "Resistor_SMD:R_0402_1005Metric" (id 2) (at 66.04 66.04 0)
