File: cm4psugroup.kicad_sch (KiCad schematic)
At the start: 0 parts

Commit message: respin
Changed lines of the file:
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@@
     (effects (font (size 1.27 1.27)) (justify left))
   )
-  (hierarchical_label "+12V_B_IN" (shape input) (at 82.55 121.92 180)
+  (hierarchical_label "+12V_IN" (shape input) (at 82.55 121.92 180)
     (effects (font (size 1.27 1.27)) (justify right))
   )
-  (hierarchical_label "CONTROL_+3.3V" (shape input) (at 170.18 81.28 180)
+  (hierarchical_label "+3.3V_CONTROL" (shape input) (at 170.18 81.28 180)
     (effects (font (size 1.27 1.27)) (justify right))
   )
@@
     (effects (font (size 1.27 1.27)) (justify right))
   )
-  (hierarchical_label "CONTROL_+3.3V" (shape input) (at 170.18 124.46 180)
+  (hierarchical_label "+3.3V_CONTROL" (shape input) (at 170.18 124.46 180)
     (effects (font (size 1.27 1.27)) (justify right))
   )
-  (hierarchical_label "+12V_A_IN" (shape input) (at 82.55 78.74 180)
+  (hierarchical_label "+12V_IN" (shape input) (at 82.55 78.74 180)
     (effects (font (size 1.27 1.27)) (justify right))
   )
@@
   (symbol (lib_id "power:GND") (at 173.99 99.06 0) (mirror y) (unit 1)
     (in_bom yes) (on_board yes) (fields_autoplaced)
-    (property "Reference" "#PWR026" (id 0) (at 173.99 105.41 0)
+    (property "Reference" "#PWR027" (id 0) (at 173.99 105.41 0)
       (effects (font (size 1.27 1.27)) hide)
     )
@@
   (symbol (lib_id "power:GND") (at 173.99 142.24 0) (mirror y) (unit 1)
     (in_bom yes) (on_board yes) (fields_autoplaced)
-    (property "Reference" "#PWR027" (id 0) (at 173.99 148.59 0)
+    (property "Reference" "#PWR028" (id 0) (at 173.99 148.59 0)
       (effects (font (size 1.27 1.27)) hide)
     )
