File: cm4psumon.kicad_sch (KiCad schematic)
At the start: 4 parts, among them U9 INA260

Commit message: board refresh
Parts:
- renumbered C14 to C12, C15 to C13, U9 to U8
Changed lines of the file:
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@@
   (symbol (lib_id "Sensor_I2C_TI:INA260") (at 125.73 67.31 0) (mirror y)
     (in_bom yes) (on_board yes)
-    (property "Reference" "U9" (id 0) (at 120.015 58.42 0))
+    (property "Reference" "U8" (id 0) (at 120.015 58.42 0))
     (property "Value" "INA260" (id 1) (at 131.445 76.2 0))
     (property "Footprint" "Sensor_I2C_TI:TSSOP-16_4.4x5mm_P0.65mm_pin1" (id 2) (at 124.46 99.06 0)
@@
   (symbol (lib_id "power:GND") (at 125.73 90.17 0)
     (in_bom yes) (on_board yes)
-    (property "Reference" "#PWR025" (id 0) (at 125.73 96.52 0)
+    (property "Reference" "#PWR023" (id 0) (at 125.73 96.52 0)
       (effects (font (size 1.27 1.27)) hide)
     )
@@
   (symbol (lib_id "power:GND") (at 69.85 68.58 0)
     (in_bom yes) (on_board yes) (fields_autoplaced)
-    (property "Reference" "#PWR024" (id 0) (at 69.85 74.93 0)
+    (property "Reference" "#PWR022" (id 0) (at 69.85 74.93 0)
       (effects (font (size 1.27 1.27)) hide)
     )
@@
   (symbol (lib_id "Device:C_Small") (at 69.85 58.42 0)
     (in_bom yes) (on_board yes) (fields_autoplaced)
-    (property "Reference" "C15" (id 0) (at 72.39 57.1562 0)
+    (property "Reference" "C13" (id 0) (at 72.39 57.1562 0)
       (effects (font (size 1.27 1.27)) (justify left))
     )
@@
   (symbol (lib_id "Device:C_Small") (at 58.42 58.42 0)
     (in_bom yes) (on_board yes) (fields_autoplaced)
-    (property "Reference" "C14" (id 0) (at 60.96 57.1562 0)
+    (property "Reference" "C12" (id 0) (at 60.96 57.1562 0)
       (effects (font (size 1.27 1.27)) (justify left))
     )
