File: cm4sensors.kicad_sch (KiCad schematic)
At the start: 22 parts, among them J3 TSM-102-01-L-SV, J4 TSM-102-01-L-SV, U10 MCP9808T-E_MC, U11 ADS7142IRUGR, U12 MCP9808T-E_MC

Commit message: board refresh
Parts:
- renumbered C16 to C14, C17 to C15, C18 to C16, C19 to C17, C20 to C18, C21 to C19, C22 to C20, C23 to C21, R32 to R35, R33 to R36, R34 to R37, R35 to R38, R36 to R39, R37 to R40, R38 to R41, R39 to R42, R40 to R43, U11 to U10, U12 to U11, U10 to U9
Changed lines of the file:
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@@
   (symbol (lib_id "Device:C_Small") (at 137.795 147.32 0) (unit 1)
     (in_bom yes) (on_board yes) (fields_autoplaced)
-    (property "Reference" "C20" (id 0) (at 140.97 146.0562 0)
+    (property "Reference" "C18" (id 0) (at 140.97 146.0562 0)
       (effects (font (size 1.27 1.27)) (justify left))
     )
@@
   (symbol (lib_id "Sensor_I2C_Microchip:MCP9808T-E_MC") (at 215.265 85.09 0) (mirror y) (unit 1)
     (in_bom yes) (on_board yes)
-    (property "Reference" "U12" (id 0) (at 205.105 73.66 0)
+    (property "Reference" "U11" (id 0) (at 205.105 73.66 0)
       (effects (font (size 1.27 1.27)) (justify left))
     )
@@
   (symbol (lib_id "power:GND") (at 121.285 100.33 0) (unit 1)
     (in_bom yes) (on_board yes) (fields_autoplaced)
-    (property "Reference" "#PWR029" (id 0) (at 121.285 106.68 0)
+    (property "Reference" "#PWR027" (id 0) (at 121.285 106.68 0)
       (effects (font (size 1.27 1.27)) hide)
     )
@@
   (symbol (lib_id "Device:R_Small") (at 151.765 147.32 0) (unit 1)
     (in_bom yes) (on_board yes) (fields_autoplaced)
-    (property "Reference" "R36" (id 0) (at 153.67 146.0499 0)
+    (property "Reference" "R39" (id 0) (at 153.67 146.0499 0)
       (effects (font (size 1.27 1.27)) (justify left))
     )
@@
   (symbol (lib_id "power:GND") (at 197.485 101.6 0) (mirror y) (unit 1)
     (in_bom yes) (on_board yes)
-    (property "Reference" "#PWR032" (id 0) (at 197.485 107.95 0)
+    (property "Reference" "#PWR030" (id 0) (at 197.485 107.95 0)
       (effects (font (size 1.27 1.27)) hide)
     )
@@
   (symbol (lib_id "Device:C_Small") (at 51.435 68.58 0) (mirror y) (unit 1)
     (in_bom yes) (on_board yes) (fields_autoplaced)
-    (property "Reference" "C18" (id 0) (at 48.895 67.31 0)
+    (property "Reference" "C16" (id 0) (at 48.895 67.31 0)
       (effects (font (size 1.27 1.27)) (justify left))
     )
@@
   (symbol (lib_name "MCP9808T-E_MC_1") (lib_id "Sensor_I2C_Microchip:MCP9808T-E_MC") (at 84.455 83.82 0) (mirror y) (unit 1)
     (in_bom yes) (on_board yes)
-    (property "Reference" "U10" (id 0) (at 74.295 72.39 0)
+    (property "Reference" "U9" (id 0) (at 74.295 72.39 0)
       (effects (font (size 1.27 1.27)) (justify left))
     )
@@
   (symbol (lib_id "Analog_ADC_TI:ADS7142IRUGR") (at 107.95 149.225 0) (unit 1)
     (in_bom yes) (on_board yes)
-    (property "Reference" "U11" (id 0) (at 88.9 132.715 0)
+    (property "Reference" "U10" (id 0) (at 88.9 132.715 0)
       (effects (font (size 1.524 1.524)))
     )
@@
   (symbol (lib_id "Device:C_Small") (at 182.245 69.85 0) (mirror y) (unit 1)
     (in_bom yes) (on_board yes) (fields_autoplaced)
-    (property "Reference" "C23" (id 0) (at 179.705 68.58 0)
+    (property "Reference" "C21" (id 0) (at 179.705 68.58 0)
       (effects (font (size 1.27 1.27)) (justify left))
     )
@@
   (symbol (lib_id "power:GND") (at 40.005 76.2 0) (mirror y) (unit 1)
     (in_bom yes) (on_board yes)
-    (property "Reference" "#PWR026" (id 0) (at 40.005 82.55 0)
+    (property "Reference" "#PWR024" (id 0) (at 40.005 82.55 0)
       (effects (font (size 1.27 1.27)) hide)
     )
@@
   (symbol (lib_id "Device:R_Small") (at 245.745 90.17 90) (unit 1)
     (in_bom yes) (on_board yes)
-    (property "Reference" "R39" (id 0) (at 240.665 88.9 90))
+    (property "Reference" "R42" (id 0) (at 240.665 88.9 90))
     (property "Value" "1k" (id 1) (at 249.555 88.9 90))
     (property "Footprint" "Resistor_SMD:R_0402_1005Metric" (id 2) (at 245.745 90.17 0)
@@
   (symbol (lib_id "Device:R_Small") (at 245.745 92.71 90) (unit 1)
     (in_bom yes) (on_board yes)
-    (property "Reference" "R40" (id 0) (at 240.665 91.44 90))
+    (property "Reference" "R43" (id 0) (at 240.665 91.44 90))
     (property "Value" "1k" (id 1) (at 249.555 91.44 90))
     (property "Footprint" "Resistor_SMD:R_0402_1005Metric" (id 2) (at 245.745 92.71 0)
@@
   (symbol (lib_id "power:GND") (at 170.815 77.47 0) (mirror y) (unit 1)
     (in_bom yes) (on_board yes)
-    (property "Reference" "#PWR031" (id 0) (at 170.815 83.82 0)
+    (property "Reference" "#PWR029" (id 0) (at 170.815 83.82 0)
       (effects (font (size 1.27 1.27)) hide)
     )
@@
   (symbol (lib_id "Device:R_Small") (at 114.935 86.36 90) (unit 1)
     (in_bom yes) (on_board yes)
-    (property "Reference" "R33" (id 0) (at 109.855 85.09 90))
+    (property "Reference" "R36" (id 0) (at 109.855 85.09 90))
     (property "Value" "1k" (id 1) (at 118.745 85.09 90))
     (property "Footprint" "Resistor_SMD:R_0402_1005Metric" (id 2) (at 114.935 86.36 0)
@@
   (symbol (lib_id "power:GND") (at 252.095 101.6 0) (mirror y) (unit 1)
     (in_bom yes) (on_board yes)
-    (property "Reference" "#PWR033" (id 0) (at 252.095 107.95 0)
+    (property "Reference" "#PWR031" (id 0) (at 252.095 107.95 0)
       (effects (font (size 1.27 1.27)) hide)
     )
@@
   (symbol (lib_id "Device:C_Small") (at 137.795 167.64 0) (unit 1)
     (in_bom yes) (on_board yes) (fields_autoplaced)
-    (property "Reference" "C21" (id 0) (at 140.97 166.3762 0)
+    (property "Reference" "C19" (id 0) (at 140.97 166.3762 0)
       (effects (font (size 1.27 1.27)) (justify left))
     )
@@
   (symbol (lib_id "Device:C_Small") (at 48.26 137.16 0) (unit 1)
     (in_bom yes) (on_board yes) (fields_autoplaced)
-    (property "Reference" "C17" (id 0) (at 51.435 135.8962 0)
+    (property "Reference" "C15" (id 0) (at 51.435 135.8962 0)
       (effects (font (size 1.27 1.27)) (justify left))
     )
@@
   (symbol (lib_id "Device:R_Small") (at 245.745 87.63 90) (unit 1)
     (in_bom yes) (on_board yes)
-    (property "Reference" "R38" (id 0) (at 240.665 86.36 90))
+    (property "Reference" "R41" (id 0) (at 240.665 86.36 90))
     (property "Value" "1k" (id 1) (at 249.555 86.36 90))
     (property "Footprint" "Resistor_SMD:R_0402_1005Metric" (id 2) (at 245.745 87.63 0)
@@
   (symbol (lib_id "Device:R_Small") (at 151.765 167.64 0) (unit 1)
     (in_bom yes) (on_board yes) (fields_autoplaced)
-    (property "Reference" "R37" (id 0) (at 153.67 166.3699 0)
+    (property "Reference" "R40" (id 0) (at 153.67 166.3699 0)
       (effects (font (size 1.27 1.27)) (justify left))
     )
@@
   (symbol (lib_id "power:GND") (at 164.465 177.165 0) (unit 1)
     (in_bom yes) (on_board yes) (fields_autoplaced)
-    (property "Reference" "#PWR030" (id 0) (at 164.465 183.515 0)
+    (property "Reference" "#PWR028" (id 0) (at 164.465 183.515 0)
       (effects (font (size 1.27 1.27)) hide)
     )
@@
   (symbol (lib_id "Device:R_Small") (at 69.215 137.16 0) (unit 1)
     (in_bom yes) (on_board yes) (fields_autoplaced)
-    (property "Reference" "R32" (id 0) (at 71.12 135.8899 0)
+    (property "Reference" "R35" (id 0) (at 71.12 135.8899 0)
       (effects (font (size 1.27 1.27)) (justify left))
     )
@@
   (symbol (lib_id "power:GND") (at 48.26 177.165 0) (unit 1)
     (in_bom yes) (on_board yes) (fields_autoplaced)
-    (property "Reference" "#PWR027" (id 0) (at 48.26 183.515 0)
+    (property "Reference" "#PWR025" (id 0) (at 48.26 183.515 0)
       (effects (font (size 1.27 1.27)) hide)
     )
@@
   (symbol (lib_id "Device:R_Small") (at 114.935 91.44 90) (unit 1)
     (in_bom yes) (on_board yes)
-    (property "Reference" "R35" (id 0) (at 109.855 90.17 90))
+    (property "Reference" "R38" (id 0) (at 109.855 90.17 90))
     (property "Value" "1k" (id 1) (at 118.745 90.17 90))
     (property "Footprint" "Resistor_SMD:R_0402_1005Metric" (id 2) (at 114.935 91.44 0)
@@
   (symbol (lib_id "Device:C_Small") (at 40.005 68.58 0) (mirror y) (unit 1)
     (in_bom yes) (on_board yes) (fields_autoplaced)
-    (property "Reference" "C16" (id 0) (at 37.465 67.31 0)
+    (property "Reference" "C14" (id 0) (at 37.465 67.31 0)
       (effects (font (size 1.27 1.27)) (justify left))
     )
@@
   (symbol (lib_id "Device:C_Small") (at 170.815 69.85 0) (mirror y) (unit 1)
     (in_bom yes) (on_board yes) (fields_autoplaced)
-    (property "Reference" "C22" (id 0) (at 168.275 68.58 0)
+    (property "Reference" "C20" (id 0) (at 168.275 68.58 0)
       (effects (font (size 1.27 1.27)) (justify left))
     )
@@
   (symbol (lib_id "Device:C_Small") (at 58.42 137.16 0) (unit 1)
     (in_bom yes) (on_board yes) (fields_autoplaced)
-    (property "Reference" "C19" (id 0) (at 61.595 135.8962 0)
+    (property "Reference" "C17" (id 0) (at 61.595 135.8962 0)
       (effects (font (size 1.27 1.27)) (justify left))
     )
@@
   (symbol (lib_id "power:GND") (at 66.675 100.33 0) (unit 1)
     (in_bom yes) (on_board yes) (fields_autoplaced)
-    (property "Reference" "#PWR028" (id 0) (at 66.675 106.68 0)
+    (property "Reference" "#PWR026" (id 0) (at 66.675 106.68 0)
       (effects (font (size 1.27 1.27)) hide)
     )
@@
   (symbol (lib_id "Device:R_Small") (at 114.935 88.9 90) (unit 1)
     (in_bom yes) (on_board yes)
-    (property "Reference" "R34" (id 0) (at 109.855 87.63 90))
+    (property "Reference" "R37" (id 0) (at 109.855 87.63 90))
     (property "Value" "1k" (id 1) (at 118.745 87.63 90))
     (property "Footprint" "Resistor_SMD:R_0402_1005Metric" (id 2) (at 114.935 88.9 0)

Commit message: work on control logic
Parts:
- renumbered R35 to R37, R36 to R38, R37 to R39, R38 to R40, R39 to R41, R40 to R42, R41 to R43, R42 to R44, R43 to R45
Changed lines of the file:
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@@
   (symbol (lib_id "Device:R_Small") (at 151.765 147.32 0) (unit 1)
     (in_bom yes) (on_board yes) (fields_autoplaced)
-    (property "Reference" "R39" (id 0) (at 153.67 146.0499 0)
+    (property "Reference" "R41" (id 0) (at 153.67 146.0499 0)
       (effects (font (size 1.27 1.27)) (justify left))
     )
@@
   (symbol (lib_id "Device:R_Small") (at 245.745 90.17 90) (unit 1)
     (in_bom yes) (on_board yes)
-    (property "Reference" "R42" (id 0) (at 240.665 88.9 90))
+    (property "Reference" "R44" (id 0) (at 240.665 88.9 90))
     (property "Value" "1k" (id 1) (at 249.555 88.9 90))
     (property "Footprint" "Resistor_SMD:R_0402_1005Metric" (id 2) (at 245.745 90.17 0)
@@
   (symbol (lib_id "Device:R_Small") (at 245.745 92.71 90) (unit 1)
     (in_bom yes) (on_board yes)
-    (property "Reference" "R43" (id 0) (at 240.665 91.44 90))
+    (property "Reference" "R45" (id 0) (at 240.665 91.44 90))
     (property "Value" "1k" (id 1) (at 249.555 91.44 90))
     (property "Footprint" "Resistor_SMD:R_0402_1005Metric" (id 2) (at 245.745 92.71 0)
@@
   (symbol (lib_id "Device:R_Small") (at 114.935 86.36 90) (unit 1)
     (in_bom yes) (on_board yes)
-    (property "Reference" "R36" (id 0) (at 109.855 85.09 90))
+    (property "Reference" "R38" (id 0) (at 109.855 85.09 90))
     (property "Value" "1k" (id 1) (at 118.745 85.09 90))
     (property "Footprint" "Resistor_SMD:R_0402_1005Metric" (id 2) (at 114.935 86.36 0)
@@
   (symbol (lib_id "Device:R_Small") (at 245.745 87.63 90) (unit 1)
     (in_bom yes) (on_board yes)
-    (property "Reference" "R41" (id 0) (at 240.665 86.36 90))
+    (property "Reference" "R43" (id 0) (at 240.665 86.36 90))
     (property "Value" "1k" (id 1) (at 249.555 86.36 90))
     (property "Footprint" "Resistor_SMD:R_0402_1005Metric" (id 2) (at 245.745 87.63 0)
@@
   (symbol (lib_id "Device:R_Small") (at 151.765 167.64 0) (unit 1)
     (in_bom yes) (on_board yes) (fields_autoplaced)
-    (property "Reference" "R40" (id 0) (at 153.67 166.3699 0)
+    (property "Reference" "R42" (id 0) (at 153.67 166.3699 0)
       (effects (font (size 1.27 1.27)) (justify left))
     )
@@
   (symbol (lib_id "Device:R_Small") (at 69.215 137.16 0) (unit 1)
     (in_bom yes) (on_board yes) (fields_autoplaced)
-    (property "Reference" "R35" (id 0) (at 71.12 135.8899 0)
+    (property "Reference" "R37" (id 0) (at 71.12 135.8899 0)
       (effects (font (size 1.27 1.27)) (justify left))
     )
@@
   (symbol (lib_id "Device:R_Small") (at 114.935 91.44 90) (unit 1)
     (in_bom yes) (on_board yes)
-    (property "Reference" "R38" (id 0) (at 109.855 90.17 90))
+    (property "Reference" "R40" (id 0) (at 109.855 90.17 90))
     (property "Value" "1k" (id 1) (at 118.745 90.17 90))
     (property "Footprint" "Resistor_SMD:R_0402_1005Metric" (id 2) (at 114.935 91.44 0)
@@
   (symbol (lib_id "Device:R_Small") (at 114.935 88.9 90) (unit 1)
     (in_bom yes) (on_board yes)
-    (property "Reference" "R37" (id 0) (at 109.855 87.63 90))
+    (property "Reference" "R39" (id 0) (at 109.855 87.63 90))
     (property "Value" "1k" (id 1) (at 118.745 87.63 90))
     (property "Footprint" "Resistor_SMD:R_0402_1005Metric" (id 2) (at 114.935 88.9 0)
