File: fruit.kicad_sch (KiCad schematic)
At the start: 7 parts, among them J1 PCB_Edge_PCI_Express_x4_Salmo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

Commit message: work on control logic
Parts:
- J1: footprint Connector_PCIe_MyOwn:BUS_PCIexpress_x4_Salmonberry_reduced_shoulders -> Connector_PCIe_MyOwn:BUS_PCIexpress_x4_Salmonberry
Connections:
- net GND: no longer J1.B12 (GND)
- new net ~{PANIC}: J1.B12 (~{PANIC1})
Other:
- sheet Fruit renamed CM4
- sheet CM4 ports: added ~{I2C_RESET_1}, ~{INT_BACKPLANE}; removed none
- note added: "Connector"
- note added: "Salmonberry Pi, Fruit \ 'früt \ CM4"
- note removed: "Mechanical"
- note removed: "Salmonberry Pi, Fruit \ 'früt \"

Commit message: work on control logic
Parts:
- added R? (x2): 10k, Resistor_SMD:R_0402_1005Metric, symbol Device:R_Small
- J1: footprint Connector_PCIe_MyOwn:BUS_PCIexpress_x4_Salmonberry -> Connector_PCIe_MyOwn:BUS_PCIexpress_x4_Salmonberry_reduced_shoulders
Connections:
- net GND: now also R?.2, R?.2
- net at J1.A11 (SWD): now also R?.1
- net at J1.A9 (SWCLK): now also R?.1
- no-connect marks 2 -> 0
Changed lines of the file:
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@@
     (comment 2 "CERN-OHL-W v2 or later")
   )
-  (no_connect (at 69.85 104.14))
-  (no_connect (at 69.85 106.68))
+  (junction (at 55.88 106.68) (diameter 0) (color 0 0 0 0)
+  )
+  (junction (at 55.88 149.86) (diameter 0) (color 0 0 0 0)
+  )
   (wire (pts (xy 118.11 86.36) (xy 97.79 86.36))
     (stroke (width 0) (type default) (color 0 0 0 0))
   )
+  (wire (pts (xy 55.88 104.14) (xy 60.96 104.14))
+    (stroke (width 0) (type default) (color 0 0 0 0))
+  )
   (wire (pts (xy 45.72 76.2) (xy 69.85 76.2))
+    (stroke (width 0) (type default) (color 0 0 0 0))
+  )
+  (wire (pts (xy 60.96 106.68) (xy 55.88 106.68))
+    (stroke (width 0) (type default) (color 0 0 0 0))
+  )
+  (wire (pts (xy 66.04 104.14) (xy 69.85 104.14))
     (stroke (width 0) (type default) (color 0 0 0 0))
   )
@@
     (stroke (width 0) (type default) (color 0 0 0 0))
   )
+  (wire (pts (xy 69.85 106.68) (xy 66.04 106.68))
+    (stroke (width 0) (type default) (color 0 0 0 0))
+  )
   (wire (pts (xy 118.11 78.74) (xy 97.79 78.74))
     (stroke (width 0) (type default) (color 0 0 0 0))
@@
     (stroke (width 0) (type default) (color 0 0 0 0))
   )
-  (wire (pts (xy 59.69 149.86) (xy 59.69 157.48))
+  (wire (pts (xy 55.88 149.86) (xy 55.88 157.48))
+    (stroke (width 0) (type default) (color 0 0 0 0))
+  )
+  (wire (pts (xy 55.88 106.68) (xy 55.88 104.14))
     (stroke (width 0) (type default) (color 0 0 0 0))
   )
@@
     (stroke (width 0) (type default) (color 0 0 0 0))
   )
-  (wire (pts (xy 69.85 149.86) (xy 59.69 149.86))
+  (wire (pts (xy 69.85 149.86) (xy 55.88 149.86))
     (stroke (width 0) (type default) (color 0 0 0 0))
   )
@@
   )
   (wire (pts (xy 118.11 83.82) (xy 97.79 83.82))
+    (stroke (width 0) (type default) (color 0 0 0 0))
+  )
+  (wire (pts (xy 55.88 149.86) (xy 55.88 106.68))
     (stroke (width 0) (type default) (color 0 0 0 0))
   )
@@
   (label "+3.3V_CONTROL" (at 190.5 73.66 0)
     (effects (font (size 1.27 1.27)) (justify left bottom))
+  )
+  (symbol (lib_id "Device:R_Small") (at 63.5 106.68 270) (unit 1)
+    (in_bom yes) (on_board yes)
+    (property "Reference" "R?" (id 0) (at 60.96 105.41 90)
+      (effects (font (size 1.27 1.27)) (justify right))
+    )
+    (property "Value" "10k" (id 1) (at 66.04 105.41 90)
+      (effects (font (size 1.27 1.27)) (justify left))
+    )
+    (property "Footprint" "Resistor_SMD:R_0402_1005Metric" (id 2) (at 63.5 106.68 0)
+      (effects (font (size 1.27 1.27)) hide)
+    )
+    (property "Datasheet" "~" (id 3) (at 63.5 106.68 0)
+      (effects (font (size 1.27 1.27)) hide)
+    )
+    (pin "1")
+    (pin "2")
   )
   (symbol (lib_id "Connector_PCIe_MyOwn:PCB_Edge_PCI_Express_x4_Salmonberry") (at 69.85 68.58 0) (unit 1)
@@
     (property "Reference" "J1" (id 0) (at 74.93 64.77 0))
     (property "Value" "PCB_Edge_PCI_Express_x4_Salmonberry" (id 1) (at 85.09 156.21 0))
-    (property "Footprint" "Connector_PCIe_MyOwn:BUS_PCIexpress_x4_Salmonberry" (id 2) (at 85.09 163.83 0)
+    (property "Footprint" "Connector_PCIe_MyOwn:BUS_PCIexpress_x4_Salmonberry_reduced_shoulders" (id 2) (at 85.09 163.83 0)
       (effects (font (size 1.27 1.27)) hide)
     )
@@
     )
   )
-  (symbol (lib_id "power:GND") (at 59.69 157.48 0) (unit 1)
+  (symbol (lib_id "power:GND") (at 55.88 157.48 0) (unit 1)
     (in_bom yes) (on_board yes) (fields_autoplaced)
-    (property "Reference" "#PWR01" (id 0) (at 59.69 163.83 0)
-      (effects (font (size 1.27 1.27)) hide)
-    )
-    (property "Value" "GND" (id 1) (at 59.69 162.56 0))
-    (property "Footprint" "" (id 2) (at 59.69 157.48 0)
-      (effects (font (size 1.27 1.27)) hide)
-    )
-    (property "Datasheet" "" (id 3) (at 59.69 157.48 0)
+    (property "Reference" "#PWR01" (id 0) (at 55.88 163.83 0)
+      (effects (font (size 1.27 1.27)) hide)
+    )
+    (property "Value" "GND" (id 1) (at 55.88 162.56 0))
+    (property "Footprint" "" (id 2) (at 55.88 157.48 0)
+      (effects (font (size 1.27 1.27)) hide)
+    )
+    (property "Datasheet" "" (id 3) (at 55.88 157.48 0)
       (effects (font (size 1.27 1.27)) hide)
     )
@@
       (effects (font (size 1.27 1.27)) hide)
     )
+  )
+  (symbol (lib_id "Device:R_Small") (at 63.5 104.14 270) (unit 1)
+    (in_bom yes) (on_board yes)
+    (property "Reference" "R?" (id 0) (at 60.96 102.87 90)
+      (effects (font (size 1.27 1.27)) (justify right))
+    )
+    (property "Value" "10k" (id 1) (at 66.04 102.87 90)
+      (effects (font (size 1.27 1.27)) (justify left))
+    )
+    (property "Footprint" "Resistor_SMD:R_0402_1005Metric" (id 2) (at 63.5 104.14 0)
+      (effects (font (size 1.27 1.27)) hide)
+    )
+    (property "Datasheet" "~" (id 3) (at 63.5 104.14 0)
+      (effects (font (size 1.27 1.27)) hide)
+    )
+    (pin "1")
+    (pin "2")
   )
   (symbol (lib_id "Mechanical_CoolingBlock:53-61mm_NorthBridge_45deg_arms") (at 104.775 180.34 0) (unit 1)
@@
     )
     (path "/0ad88b14-75ca-4fe9-9bb6-f5d58fe3e7f9"
-      (reference "J1") (unit 1) (value "PCB_Edge_PCI_Express_x4_Salmonberry") (footprint "Connector_PCIe_MyOwn:BUS_PCIexpress_x4_Salmonberry")
+      (reference "J1") (unit 1) (value "PCB_Edge_PCI_Express_x4_Salmonberry") (footprint "Connector_PCIe_MyOwn:BUS_PCIexpress_x4_Salmonberry_reduced_shoulders")
     )
     (path "/c9dd42ab-5b09-45b1-aea9-aad38fed4868/4f5f12fb-6c4a-4c4e-bd75-97c375c6157a/1e957c1a-1b39-44d9-8d63-adc9bfb3c01d"
@@
       (reference "R77") (unit 1) (value "50R") (footprint "Resistor_SMD:R_0402_1005Metric")
     )
+    (path "/0a6e002a-09fe-41ec-b21b-865fe65e2dda"
+      (reference "R?") (unit 1) (value "10k") (footprint "Resistor_SMD:R_0402_1005Metric")
+    )
+    (path "/de81afff-4c8f-4e82-9798-f73bbc52226b"
+      (reference "R?") (unit 1) (value "10k") (footprint "Resistor_SMD:R_0402_1005Metric")
+    )
     (path "/c9dd42ab-5b09-45b1-aea9-aad38fed4868/af8eef5a-1d65-4630-994e-2dc09fa9cc79/f4eb04ea-f65a-457e-ab30-6a8beed169b8/d7a4ed94-9fd3-457c-8e59-d187492c288c"

Commit message: work on control logic
Parts:
- gave numbers to parts that had none: 2
