File: fruit.kicad_pcb (KiCad board)
At the start: 4 copper layers, 161.6 x 100 mm, 210 parts, among them J1 PCB_Edge_PCI_Express_x4_Salmo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, J2 2086581051, J3 TSM-102-01-L-SV, J4 TSM-102-01-L-SV, J5 MEM2067-02-180-00-A_REVB, J6 USB4110-GF-A, J7 USB4110-GF-A, J8 1-2199119-6, Q1 MMBT2222AM3T5G, U1 INA260, U10 MCP9808T-E_MC, U11 ADS7142IRUGR, U12 MCP9808T-E_MC, U13 LM3525M-H_NPOB, U14 USB3740B-AI2, U15 AP22653FDZ-7, U16 AP64501SP-13, U17 AP64501SP-13, U2 PCA9671BS,118, U3 PCA9671BS,118, U4 SN74LVC1G04DRY, U5 SN74LVC1G07DRY, U6 PCA9641BSHP, U7 AP22653FDZ-7, U8 TPD8S009DSMR, U9 INA260

Commit message: work on control logic
Parts:
- COOLER1: value 53-61mm_NorthBridge_45deg_arms -> 53-61
- J2: value 2086581051 -> CONN_208658-1051_MOL
- J6, J7: value USB4110-GF-A -> GCT_USB4110-GF-A
- Q1: value MMBT2222AM3T5G -> SOT-723_0P85X1P25_ONS
- U11: value ADS7142IRUGR -> RUG0010A

Commit message: board refresh
Parts:
- added R20: 100k, Resistor_SMD:R_0402_1005Metric, F.Cu at (207.6, -25.9)
- added R21: 100k, Resistor_SMD:R_0402_1005Metric, F.Cu at (210.5, -27.9)
- added R22: 100k, Resistor_SMD:R_0402_1005Metric, F.Cu at (204.6, -29.9)
- added R27: 10k, Resistor_SMD:R_0402_1005Metric, F.Cu at (204.6, -27.9)
- added R28: 10k, Resistor_SMD:R_0402_1005Metric, F.Cu at (204.6, -25.9)
- added R29: 10k, Resistor_SMD:R_0402_1005Metric, F.Cu at (207.6, -27.9)
- added R30: 10k, Resistor_SMD:R_0402_1005Metric, F.Cu at (210.5, -25.9)
- added R31: 10k, Resistor_SMD:R_0402_1005Metric, F.Cu at (207.6, -29.9)
- added R32: 10k, Resistor_SMD:R_0402_1005Metric, F.Cu at (210.5, -29.9)
- COOLER1: value 53-61 -> 53-61mm_NorthBridge_45deg_arms
- J1: footprint Connector_PCIe_MyOwn:BUS_PCIexpress_x4_Salmonberry_reduced_shoulders -> Connector_PCIe_MyOwn:BUS_PCIexpress_x4_Salmonberry
- J2: value CONN_208658-1051_MOL -> 2086581051
- J6, J7: value GCT_USB4110-GF-A -> USB4110-GF-A
- Q1: value SOT-723_0P85X1P25_ONS -> MMBT2222AM3T5G
- U10: renamed from U11; value RUG0010A -> ADS7142IRUGR
- renumbered C12 to C10, C13 to C11, C14 to C12, C15 to C13, C16 to C14, C17 to C15, C18 to C16, C19 to C17, C20 to C18, C21 to C19, C22 to C20, C23 to C21, C24 to C22, C25 to C23, C26 to C24, C27 to C25, C28 to C26, C29 to C27, C30 to C28, C31 to C29, C32 to C30, C33 to C31, C34 to C32, C35 to C33, C36 to C34, C37 to C35, C38 to C36, C39 to C37, C40 to C38, C41 to C39, C42 to C40, C43 to C41, C44 to C42, C45 to C43, C47 to C45, C48 to C46, C49 to C47, C50 to C48, C51 to C49, C7 to C5, C52 to C50, C53 to C51, C54 to C52, C55 to C53, C56 to C54, C57 to C55, C58 to C56, C59 to C57, C60 to C58, C61 to C59, C8 to C6, C63 to C61, C64 to C62, C65 to C63, C66 to C64, C67 to C65, C68 to C66, C69 to C67, C70 to C68, C71 to C69, C9 to C7, C72 to C70, C73 to C71, C74 to C72, C75 to C73, C76 to C74, C77 to C75, C78 to C76, C10 to C8, C11 to C9, D6 to D1, D1 to D2, D2 to D3, D3 to D4, D4 to D5, D5 to D6, R11 to R10, R12 to R11, R13 to R12, R20 to R13, R24 to R14, R25 to R15, R26 to R16, R27 to R17, R28 to R18, R29 to R19, R22 to R2, R5 to R23, R6 to R24, R7 to R25, R8 to R26, R14 to R3, R30 to R33, R31 to R34, R32 to R35, R33 to R36, R34 to R37, R35 to R38, R36 to R39, R15 to R4, R37 to R40, R38 to R41, R39 to R42, R40 to R43, R41 to R44, R42 to R45, R43 to R46, R44 to R47, R45 to R48, R46 to R49, R16 to R5, R47 to R50, R48 to R51, R49 to R52, R50 to R53, R51 to R54, R52 to R55, R53 to R56, R54 to R57, R55 to R58, R56 to R59, R17 to R6, R57 to R60, R58 to R61, R59 to R62, R60 to R63, R61 to R64, R62 to R65, R63 to R66, R64 to R67, R65 to R68, R66 to R69, R18 to R7, R67 to R70, R68 to R71, R69 to R72, R70 to R73, R71 to R74, R72 to R75, R73 to R76, R74 to R77, R9 to R8, R10 to R9, TP3 to TP2, TP5 to TP3, TP6 to TP4, TP7 to TP5, TP8 to TP6, TP9 to TP7, TP2 to TP8, TP4 to TP9, U12 to U11, U13 to U12, U14 to U13, U15 to U14, U16 to U15, U17 to U16, U4 to U3, U5 to U4, U6 to U5, U7 to U6, U8 to U7, U9 to U8, U10 to U9
Connections:
- net /Fruit/CM4 Hirose connectors/GPIO10 renamed /CM4/CM4 Hirose connectors/GPIO10
- net /Fruit/CM4 Hirose connectors/GPIO11 renamed /CM4/CM4 Hirose connectors/GPIO11
- net /Fruit/CM4 Hirose connectors/GPIO12 renamed /CM4/CM4 Hirose connectors/GPIO12
- net /Fruit/CM4 Hirose connectors/GPIO13 renamed /CM4/CM4 Hirose connectors/GPIO13
- net /Fruit/CM4 Hirose connectors/GPIO18 renamed /CM4/CM4 Hirose connectors/GPIO18
- net /Fruit/CM4 Hirose connectors/GPIO19 renamed /CM4/CM4 Hirose connectors/GPIO19
- net /Fruit/CM4 Hirose connectors/GPIO2 renamed /CM4/CM4 Hirose connectors/GPIO2
- net /Fruit/CM4 Hirose connectors/GPIO20 renamed /CM4/CM4 Hirose connectors/GPIO20
- net /Fruit/CM4 Hirose connectors/GPIO21 renamed /CM4/CM4 Hirose connectors/GPIO21
- net /Fruit/CM4 Hirose connectors/GPIO22 renamed /CM4/CM4 Hirose connectors/GPIO22
- net /Fruit/CM4 Hirose connectors/GPIO23 renamed /CM4/CM4 Hirose connectors/GPIO23
- net /Fruit/CM4 Hirose connectors/GPIO3 renamed /CM4/CM4 Hirose connectors/GPIO3
- net /Fruit/CM4 Hirose connectors/GPIO4 renamed /CM4/CM4 Hirose connectors/GPIO4
- net /Fruit/CM4 Hirose connectors/GPIO5 renamed /CM4/CM4 Hirose connectors/GPIO5
- net /Fruit/CM4 Hirose connectors/GPIO6 renamed /CM4/CM4 Hirose connectors/GPIO6
- net /Fruit/CM4 Hirose connectors/GPIO7 renamed /CM4/CM4 Hirose connectors/GPIO7
- net /Fruit/CM4 Hirose connectors/GPIO8 renamed /CM4/CM4 Hirose connectors/GPIO8
- net /Fruit/CM4 Hirose connectors/GPIO9 renamed /CM4/CM4 Hirose connectors/GPIO9
- net /Fruit/CM4 Hirose connectors/ID_SC renamed /CM4/CM4 Hirose connectors/ID_SC
- net /Fruit/CM4 Hirose connectors/ID_SD renamed /CM4/CM4 Hirose connectors/ID_SD
- net /Fruit/CM4 Hirose connectors/~{EXTRST} renamed /CM4/CM4 Hirose connectors/~{EXTRST}
- net /Fruit/CM4 PSU/+12V_IN renamed /CM4/CM4 PSU/+12V_IN
- net /Fruit/CM4 PSU/+3.3V PSU/+3.3V_OUT renamed /CM4/CM4 PSU/+3.3V PSU/+3.3V_OUT
- net /Fruit/CM4 PSU/+3.3V_CONTROL renamed /CM4/CM4 PSU/+3.3V_CONTROL
- net /Fruit/CM4 PSU/+5V PSU/+5V_OUT renamed /CM4/CM4 PSU/+5V PSU/+5V_OUT
- net /Fruit/CM4_+5V renamed /CM4/CM4_+5V
- net /Fruit/CM4_I2C_SCL renamed /CM4/CM4_I2C_SCL
- net /Fruit/CM4_I2C_SDA renamed /CM4/CM4_I2C_SDA
- net /Fruit/CM4_OUT_+1.8V renamed /CM4/CM4_OUT_+1.8V
- net /Fruit/CM4_OUT_+3.3V renamed /CM4/CM4_OUT_+3.3V
- net /Fruit/HDMI/HDMI_+5V renamed /CM4/HDMI/HDMI_+5V
- net /Fruit/HDMICEC renamed /CM4/HDMICEC
- net /Fruit/HDMICK+ renamed /CM4/HDMICK+
- net /Fruit/HDMICK- renamed /CM4/HDMICK-
- net /Fruit/HDMID0+ renamed /CM4/HDMID0+
- net /Fruit/HDMID0- renamed /CM4/HDMID0-
- net /Fruit/HDMID1+ renamed /CM4/HDMID1+
- net /Fruit/HDMID1- renamed /CM4/HDMID1-
- net /Fruit/HDMID2+ renamed /CM4/HDMID2+
- net /Fruit/HDMID2- renamed /CM4/HDMID2-
- net /Fruit/HDMIHP renamed /CM4/HDMIHP
- net /Fruit/HDMISCL renamed /CM4/HDMISCL
- net /Fruit/HDMISDA renamed /CM4/HDMISDA
- net /Fruit/I2C GPIO1/GPIO17 renamed /CM4/I2C GPIO1/GPIO17
- net /Fruit/I2C GPIO1/I2C_A0 renamed /CM4/I2C GPIO1/I2C_A0
- net /Fruit/I2C GPIO1/I2C_A1 renamed /CM4/I2C GPIO1/I2C_A1
- net /Fruit/I2C GPIO1/I2C_A2 renamed /CM4/I2C GPIO1/I2C_A2
- net /Fruit/I2C_PING_1 renamed /CM4/I2C_PING_1
- net /Fruit/M2_1_ACTIVITY_LED renamed /CM4/M2_1_ACTIVITY_LED
- net /Fruit/PCIE_CLK+ renamed /CM4/PCIE_CLK+
- net /Fruit/PCIE_CLK- renamed /CM4/PCIE_CLK-
- net /Fruit/PCIE_RX+ renamed /CM4/PCIE_RX+
- net /Fruit/PCIE_RX- renamed /CM4/PCIE_RX-
- net /Fruit/PCIE_TX+ renamed /CM4/PCIE_TX+
- net /Fruit/PCIE_TX- renamed /CM4/PCIE_TX-
- net /Fruit/SD_CLK renamed /CM4/SD_CLK
- net /Fruit/SD_CMD renamed /CM4/SD_CMD
- net /Fruit/SD_DAT0 renamed /CM4/SD_DAT0
- net /Fruit/SD_DAT1 renamed /CM4/SD_DAT1
- net /Fruit/SD_DAT2 renamed /CM4/SD_DAT2
- net /Fruit/SD_DAT3 renamed /CM4/SD_DAT3
- net /Fruit/SD_PWR_ON renamed /CM4/SD_PWR_ON
- net /Fruit/Sensors/CM4_TEMP_A0 renamed /CM4/Sensors/CM4_TEMP_A0
- net /Fruit/Sensors/CM4_TEMP_A1 renamed /CM4/Sensors/CM4_TEMP_A1
- net /Fruit/Sensors/CM4_TEMP_A2 renamed /CM4/Sensors/CM4_TEMP_A2
- net /Fruit/Sensors/M.2_TEMP_A0 renamed /CM4/Sensors/M.2_TEMP_A0
- net /Fruit/Sensors/M.2_TEMP_A1 renamed /CM4/Sensors/M.2_TEMP_A1
- net /Fruit/Sensors/M.2_TEMP_A2 renamed /CM4/Sensors/M.2_TEMP_A2
- net /Fruit/USB 2.0 MUX/HD1+ renamed /CM4/USB 2.0 MUX/HD1+
- net /Fruit/USB 2.0 MUX/HD1- renamed /CM4/USB 2.0 MUX/HD1-
- net /Fruit/USB 2.0 MUX/HD_OTG+ renamed /CM4/USB 2.0 MUX/HD_OTG+
- net /Fruit/USB 2.0 MUX/HD_OTG- renamed /CM4/USB 2.0 MUX/HD_OTG-
- net /Fruit/USB 2.0 MUX/VBUS1 renamed /CM4/USB 2.0 MUX/VBUS1
- net /Fruit/USB 2.0 MUX/VBUS_OTG renamed /CM4/USB 2.0 MUX/VBUS_OTG
- net /Fruit/USB+ renamed /CM4/USB+
- net /Fruit/USB- renamed /CM4/USB-
- net /Fruit/USBOTG renamed /CM4/USBOTG
- net /Fruit/micro SD card/SD_VDD renamed /CM4/micro SD card/SD_VDD
- net /Fruit/~{EthLED1} renamed /CM4/~{EthLED1}
- net /Fruit/~{EthLED2} renamed /CM4/~{EthLED2}
- net /Fruit/~{EthLED3} renamed /CM4/~{EthLED3}
- net /Fruit/~{I2C_RESET_1} renamed /CM4/I2C GPIO1/~{I2C_RESET}
- net /Fruit/~{PCIE_CLK_REQ} renamed /CM4/~{PCIE_CLK_REQ}
- net /Fruit/~{PCIE_RST} renamed /CM4/~{PCIE_RST}
- net /Fruit/~{PI_Activity} renamed /CM4/~{PI_Activity}
- net /Fruit/~{PWR_LED} renamed /CM4/~{PWR_LED}
- C22 pad 1: /Fruit/CM4_+3.3V -> /CM4/CM4_+3.3V
- C25 pad 1: /Fruit/CM4_+3.3V -> /CM4/CM4_+3.3V
- C26 pad 1: /Fruit/CM4_+3.3V -> /CM4/CM4_+3.3V
- C3 pad 1: +12V -> /CM4/I2C GPIO1/+3.3V_IN
- C4 pad 1: +12V -> /CM4/I2C GPIO1/+3.3V_IN
- C5 pad 1: /Fruit/CM4_+3.3V -> /CM4/CM4_+3.3V
- C66 pad 1: /Fruit/CM4_+3.3V -> /CM4/CM4_+3.3V
- C67 pad 1: /Fruit/CM4_+3.3V -> /CM4/CM4_+3.3V
- C68 pad 1: /Fruit/CM4_+3.3V -> /CM4/CM4_+3.3V
- C69 pad 1: /Fruit/CM4_+3.3V -> /CM4/CM4_+3.3V
- C70 pad 1: /Fruit/CM4_+3.3V -> /CM4/CM4_+3.3V
- C71 pad 1: /Fruit/CM4_+3.3V -> /CM4/CM4_+3.3V
- C72 pad 1: /Fruit/CM4_+3.3V -> /CM4/CM4_+3.3V
- C73 pad 1: /Fruit/CM4_+3.3V -> /CM4/CM4_+3.3V
- C74 pad 1: /Fruit/CM4_+3.3V -> /CM4/CM4_+3.3V
- C75 pad 1: /Fruit/CM4_+3.3V -> /CM4/CM4_+3.3V
- C76 pad 1: /Fruit/CM4_+3.3V -> /CM4/CM4_+3.3V
- CM1 pad 24: /Fruit/SOFT_HALT -> /CM4/SOFT_HALT
- CM1 pad 41: /Fruit/CM4 Hirose connectors/GPIO25 -> /~{I2C_RESET}
- CM1 pad 45: /Fruit/CM4 Hirose connectors/GPIO24 -> /CM4/~{INT_CM4}
- CM1 pad 48: /Fruit/SOFT_REBOOT -> /CM4/SOFT_REBOOT
- CM1 pad 92: /Fruit/I2C_RUN_PG -> /CM4/I2C_RUN_PG
- CM1 pad 93: /Fruit/~{I2C_RPI_BOOT} -> /CM4/~{I2C_RPI_BOOT}
- CM1 pad 99: /Fruit/I2C_GLOBAL_EN -> /CM4/I2C_GLOBAL_EN
- J1 pad B12: GND -> /~{PANIC}
- J8 pad 12: /Fruit/CM4_+3.3V -> /CM4/CM4_+3.3V
- J8 pad 14: /Fruit/CM4_+3.3V -> /CM4/CM4_+3.3V
- J8 pad 16: /Fruit/CM4_+3.3V -> /CM4/CM4_+3.3V
- J8 pad 18: /Fruit/CM4_+3.3V -> /CM4/CM4_+3.3V
- J8 pad 2: /Fruit/CM4_+3.3V -> /CM4/CM4_+3.3V
- J8 pad 4: /Fruit/CM4_+3.3V -> /CM4/CM4_+3.3V
- J8 pad 70: /Fruit/CM4_+3.3V -> /CM4/CM4_+3.3V
- J8 pad 72: /Fruit/CM4_+3.3V -> /CM4/CM4_+3.3V
- J8 pad 74: /Fruit/CM4_+3.3V -> /CM4/CM4_+3.3V
- R1 pad 2: +12V -> /CM4/I2C GPIO1/+3.3V_IN
- R2 pad 2: Net-(R22-Pad2) -> Net-(R2-Pad2)
- R23 pad 1: /Fruit/I2C_SCL -> /CM4/I2C_SCL
- R24 pad 1: /Fruit/I2C_SDA -> /CM4/I2C_SDA
- R3 pad 2: /Fruit/CM4_+3.3V -> /CM4/CM4_+3.3V
- R4 pad 2: /Fruit/CM4_+3.3V -> /CM4/CM4_+3.3V
- R44 pad 1: /Fruit/CM4_+3.3V -> /CM4/CM4_+3.3V
- R5 pad 1: /Fruit/CM4_+3.3V -> /CM4/CM4_+3.3V
- R6 pad 1: /Fruit/CM4_+3.3V -> /CM4/CM4_+3.3V
- R7 pad 1: /Fruit/CM4_+3.3V -> /CM4/CM4_+3.3V
- TP10 pad 1: /Fruit/CM4_+3.3V -> /CM4/CM4_+3.3V
- TP2 pad 1: Net-(R22-Pad2) -> Net-(R2-Pad2)
- U1 pad 7: /Fruit/CM4_ALERT_+5V -> /CM4/CM4_ALERT_+5V
- U1 pad 8: /Fruit/I2C_SDA -> /CM4/I2C_SDA
- U1 pad 9: /Fruit/I2C_SCL -> /CM4/I2C_SCL
- U10 pad 7: /Fruit/I2C_SDA -> /CM4/I2C_SDA
- U10 pad 8: /Fruit/I2C_SCL -> /CM4/I2C_SCL
- U11 pad 1: /Fruit/I2C_SDA -> /CM4/I2C_SDA
- U11 pad 2: /Fruit/I2C_SCL -> /CM4/I2C_SCL
- U11 pad 3: /Fruit/M.2_TALERT -> /CM4/M.2_TALERT
- U12 pad 7: /Fruit/CM4_+3.3V -> /CM4/CM4_+3.3V
- U13 pad 5: /Fruit/CM4_+3.3V -> /CM4/CM4_+3.3V
- U15 pad 3: /Fruit/CM4_EN_+3.3V -> /CM4/CM4_EN_+3.3V
- U16 pad 3: /Fruit/CM4_EN_+5V -> /CM4/CM4_EN_+5V
- U2 pad 10: /Fruit/I2C GPIO1/GPIO10 -> /CM4/CM4_EN_+3.3V
- U2 pad 11: /Fruit/I2C GPIO1/GPIO11 -> /CM4/CM4_EN_+5V
- U2 pad 12: /Fruit/I2C GPIO1/GPIO12 -> /CM4/~{I2C_RPI_BOOT}
- U2 pad 13: /Fruit/I2C GPIO1/GPIO13 -> /CM4/I2C_GLOBAL_EN
- U2 pad 14: /Fruit/I2C GPIO1/GPIO14 -> /CM4/SOFT_REBOOT
- U2 pad 15: /Fruit/I2C GPIO1/GPIO15 -> /CM4/I2C_RUN_PG
- U2 pad 16: /Fruit/I2C GPIO1/GPIO16 -> /CM4/SOFT_HALT
- U2 pad 19: /Fruit/I2C_SCL -> /CM4/I2C GPIO1/I2C_SCL
- U2 pad 20: /Fruit/I2C_SDA -> /CM4/I2C GPIO1/I2C_SDA
- U2 pad 21: +12V -> /CM4/I2C GPIO1/+3.3V_IN
- U2 pad 4: /Fruit/I2C GPIO1/GPIO03 -> /CM4/CM4_ALERT_+3.3V
- U2 pad 5: /Fruit/I2C GPIO1/GPIO04 -> /CM4/CM4_ALERT_+5V
- U2 pad 6: /Fruit/I2C GPIO1/GPIO05 -> /CM4/CM4_TALERT
- U2 pad 7: /Fruit/I2C GPIO1/GPIO06 -> /CM4/M.2_TALERT
- U3 pad 1: unconnected-(U4-Pad1) -> unconnected-(U3-Pad1)
- U3 pad 4: Net-(R22-Pad2) -> Net-(R2-Pad2)
- U3 pad 6: /Fruit/CM4_+3.3V -> /CM4/CM4_+3.3V
- U4 pad 1: unconnected-(U5-Pad1) -> unconnected-(U4-Pad1)
- U4 pad 6: /Fruit/CM4_+3.3V -> /CM4/CM4_+3.3V
- U5 pad 11: /Fruit/I2C_SCL -> /CM4/I2C_SCL
- U5 pad 12: /Fruit/I2C_SDA -> /CM4/I2C_SDA
- U5 pad 13: unconnected-(U6-Pad13) -> /CM4/~{INT_IN}
- U5 pad 15: unconnected-(U6-Pad15) -> /~{PANIC}
- U5 pad 2: unconnected-(U6-Pad2) -> /CM4/~{I2C_RESET_1_1}
- U5 pad 5: unconnected-(U6-Pad5) -> /CM4/~{INT_CM4}
- U8 pad 14: /Fruit/CM4_+3.3V -> /CM4/CM4_+3.3V
- U8 pad 15: /Fruit/CM4_+3.3V -> /CM4/CM4_+3.3V
- U8 pad 16: /Fruit/CM4_+3.3V -> /CM4/CM4_+3.3V
- U8 pad 7: /Fruit/CM4_ALERT_+3.3V -> /CM4/CM4_ALERT_+3.3V
- U8 pad 8: /Fruit/I2C_SDA -> /CM4/I2C_SDA
- U8 pad 9: /Fruit/I2C_SCL -> /CM4/I2C_SCL
- U9 pad 1: /Fruit/I2C_SDA -> /CM4/I2C_SDA
- U9 pad 2: /Fruit/I2C_SCL -> /CM4/I2C_SCL
- U9 pad 3: /Fruit/CM4_TALERT -> /CM4/CM4_TALERT

Commit message: work on control logic
Parts:
- J1: footprint Connector_PCIe_MyOwn:BUS_PCIexpress_x4_Salmonberry -> Connector_PCIe_MyOwn:BUS_PCIexpress_x4_Salmonberry_reduced_shoulders
Changed lines of the file:
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@@
     )
   )
-  (footprint "Connector_PCIe_MyOwn:BUS_PCIexpress_x4_Salmonberry" locked (layer "B.Cu")
+  (footprint "Connector_PCIe_MyOwn:BUS_PCIexpress_x4_Salmonberry_reduced_shoulders" locked (layer "B.Cu")
     (at 163.55 33.5 -90)
     (descr "PCIexpress Bus Edge Connector x1 http://www.ritrontek.com/uploadfile/2016/1026/20161026105231124.pdf#page=70")
@@
     )
     (fp_line (start 12.45 4) (end 12.45 -2.95) (layer "Edge.Cuts") (width 0.1))
+    (fp_line (start 33.65 -2.95) (end 33.15 -3.45) (layer "Edge.Cuts") (width 0.1))
+    (fp_line (start 10.55 -2.95) (end 10.05 -3.45) (layer "Edge.Cuts") (width 0.1))
+    (fp_line (start -0.65 1.95) (end -0.65 -2.95) (layer "Edge.Cuts") (width 0.1))
+    (fp_line (start -0.65 -2.95) (end -0.15 -3.45) (layer "Edge.Cuts") (width 0.1))
+    (fp_line (start 12.95 -3.45) (end 33.15 -3.45) (layer "Edge.Cuts") (width 0.1))
     (fp_line (start 12.45 -2.95) (end 12.95 -3.45) (layer "Edge.Cuts") (width 0.1))
-    (fp_line (start -0.65 4.95) (end -0.65 -2.95) (layer "Edge.Cuts") (width 0.1))
-    (fp_line (start 10.55 -2.95) (end 10.05 -3.45) (layer "Edge.Cuts") (width 0.1))
-    (fp_line (start 12.95 -3.45) (end 33.15 -3.45) (layer "Edge.Cuts") (width 0.1))
-    (fp_line (start -0.65 -2.95) (end -0.15 -3.45) (layer "Edge.Cuts") (width 0.1))
-    (fp_line (start 33.65 4.95) (end 33.65 -2.95) (layer "Edge.Cuts") (width 0.1))
+    (fp_line (start 33.65 1.95) (end 33.65 -2.95) (layer "Edge.Cuts") (width 0.1))
+    (fp_line (start 10.55 4) (end 10.55 -2.95) (layer "Edge.Cuts") (width 0.1))
     (fp_line (start -0.15 -3.45) (end 10.05 -3.45) (layer "Edge.Cuts") (width 0.1))
-    (fp_line (start 33.65 -2.95) (end 33.15 -3.45) (layer "Edge.Cuts") (width 0.1))
-    (fp_line (start 10.55 4) (end 10.55 -2.95) (layer "Edge.Cuts") (width 0.1))
     (fp_arc (start 12.45 4) (mid 11.5 4.95) (end 10.55 4) (layer "Edge.Cuts") (width 0.1))
+    (fp_line (start -1.15 5.45) (end -1.15 -3.95) (layer "B.CrtYd") (width 0.05))
+    (fp_line (start -1.15 5.45) (end 34.15 5.45) (layer "B.CrtYd") (width 0.05))
     (fp_line (start 34.15 -3.95) (end 34.15 5.45) (layer "B.CrtYd") (width 0.05))
-    (fp_line (start -1.15 5.45) (end 34.15 5.45) (layer "B.CrtYd") (width 0.05))
-    (fp_line (start -1.15 5.45) (end -1.15 -3.95) (layer "B.CrtYd") (width 0.05))
     (fp_line (start 34.15 -3.95) (end -1.15 -3.95) (layer "B.CrtYd") (width 0.05))
     (pad "A1" connect rect locked (at 0 0.55 270) (size 0.7 3.2) (layers "F.Cu" "F.Mask")

Commit message: work on control logic
Parts:
- added R1: 10k, Resistor_SMD:R_0402_1005Metric, F.Cu at (208.5, -21.8)
- added R2: 10k, Resistor_SMD:R_0402_1005Metric, F.Cu at (205.6, -21.8)
- renumbered R8 to R10, R9 to R11, R10 to R12, R11 to R13, R12 to R14, R13 to R15, R14 to R16, R15 to R17, R16 to R18, R17 to R19, R18 to R20, R19 to R21, R20 to R22, R21 to R23, R22 to R24, R23 to R25, R24 to R26, R25 to R27, R26 to R28, R27 to R29, R1 to R3, R28 to R30, R29 to R31, R30 to R32, R31 to R33, R32 to R34, R33 to R35, R34 to R36, R35 to R37, R36 to R38, R37 to R39, R2 to R4, R38 to R40, R39 to R41, R40 to R42, R41 to R43, R42 to R44, R43 to R45, R44 to R46, R45 to R47, R46 to R48, R47 to R49, R3 to R5, R48 to R50, R49 to R51, R50 to R52, R51 to R53, R52 to R54, R53 to R55, R54 to R56, R55 to R57, R56 to R58, R57 to R59, R4 to R6, R58 to R60, R59 to R61, R60 to R62, R61 to R63, R62 to R64, R63 to R65, R64 to R66, R65 to R67, R66 to R68, R67 to R69, R5 to R7, R68 to R70, R69 to R71, R70 to R72, R71 to R73, R72 to R74, R73 to R75, R74 to R76, R75 to R77, R76 to R78, R77 to R79, R6 to R8, R7 to R9
Connections:
- J1 pad A11: unconnected-(J1-PadA11) -> Net-(J1-PadA11)
- J1 pad A9: unconnected-(J1-PadA9) -> Net-(J1-PadA9)
- R4 pad 2: Net-(R2-Pad2) -> Net-(R4-Pad2)
- TP2 pad 1: Net-(R2-Pad2) -> Net-(R4-Pad2)
- U3 pad 4: Net-(R2-Pad2) -> Net-(R4-Pad2)

Commit message: work on control logic
Parts:
- removed the C12 at (51.3, 241.7)
- removed the C13 at (60.5, 232.1)
- removed the C5 at (108.2, -41.2)
- removed the C6 at (97.2, -30.4)
- removed the R19 at (16.2, 71.9)
- removed the R2 at (97.2, -32.4)
- removed the R21 at (22.1, 69.4)
- removed the R23 at (25.1, 68.5)
- removed the R3 at (107.9, -45.2)
- removed the R4 at (97.2, -36.3)
- removed the U3 at (99.3, -45.6)
- removed the U4 at (30.9, 71.9)
- removed the U8 at (54.6, 234.4)
- added C14: 10uF, Capacitor_SMD:C_0402_1005Metric, F.Cu at (62.3, 232.6)
- added C15: 0.1uF, Capacitor_SMD:C_0402_1005Metric, F.Cu at (62.3, 234.6)
- added C7: 10uF, Capacitor_SMD:C_0402_1005Metric, F.Cu at (221.6, -44.3)
- added C8: 0.1uF, Capacitor_SMD:C_0402_1005Metric, F.Cu at (218.6, -42.3)
- added R13: 1k, Resistor_SMD:R_0402_1005Metric, F.Cu at (218.7, -44.3)
- added R14: 1k, Resistor_SMD:R_0402_1005Metric, F.Cu at (221.6, -46.2)
- added R37: 10k, Resistor_SMD:R_0402_1005Metric, F.Cu at (218.7, -46.2)
- added U5: SN74HCS244, Buffer_SMD_TI:RKS0020A, F.Cu at (214.9, -43.9)
- added U9: INA260, Sensor_I2C_TI:TSSOP-16_4.4x5mm_P0.65mm_pin1, F.Cu at (56.5, 231.9)
- moved Q1 77.6 mm to (-32.4, 124.1)
- moved R16 77.6 mm to (-33.4, 129.1)
- moved LED1 77.6 mm to (-38.9, 121.8)
- moved R15 77.6 mm to (-30.5, 128.6)
- moved R17 77.6 mm to (-29.6, 123.7)
- moved R18 77.6 mm to (-26.7, 123.7)
- moved R19 77.6 mm to (-33.3, 126.6)
- moved TP8 77.6 mm to (-36.3, 126.5)
- moved TP10 14.2 mm to (62.4, 230.1)
- moved C69 7.12 mm to (51.8, 98.1)
- moved R69 7.12 mm to (49.8, 95.2)
- moved R70 7.12 mm to (51.8, 95.2)
- moved R80 7.12 mm to (53.8, 95.2)
- moved R81 7.12 mm to (53.8, 98.1)
- renumbered C8 to C10, C9 to C11, C10 to C12, C11 to C13, C14 to C16, C15 to C17, C16 to C18, C17 to C19, C18 to C20, C19 to C21, C20 to C22, C21 to C23, C22 to C24, C23 to C25, C24 to C26, C25 to C27, C26 to C28, C27 to C29, C28 to C30, C29 to C31, C30 to C32, C31 to C33, C32 to C34, C33 to C35, C34 to C36, C35 to C37, C36 to C38, C37 to C39, C38 to C40, C39 to C41, C40 to C42, C41 to C43, C42 to C44, C43 to C45, C45 to C47, C46 to C48, C47 to C49, C48 to C50, C49 to C51, C50 to C52, C51 to C53, C52 to C54, C53 to C55, C54 to C56, C55 to C57, C56 to C58, C57 to C59, C58 to C60, C59 to C61, C61 to C63, C62 to C64, C63 to C65, C64 to C66, C65 to C67, C66 to C68, C67 to C69, C68 to C70, C69 to C71, C70 to C72, C71 to C73, C72 to C74, C73 to C75, C74 to C76, C75 to C77, C76 to C78, C7 to C9, R13 to R15, R14 to R16, R15 to R17, R16 to R18, R17 to R19, R18 to R20, R19 to R21, R20 to R22, R21 to R23, R25 to R24, R26 to R25, R27 to R26, R28 to R27, R29 to R28, R30 to R29, R31 to R30, R32 to R31, R33 to R32, R34 to R33, R22 to R34, R23 to R35, R24 to R36, R35 to R38, R36 to R39, R37 to R40, R38 to R41, R39 to R42, R40 to R43, R41 to R44, R42 to R45, R43 to R46, R44 to R47, R45 to R48, R46 to R49, R47 to R50, R48 to R51, R49 to R52, R50 to R53, R51 to R54, R52 to R55, R53 to R56, R54 to R57, R55 to R58, R56 to R59, R57 to R60, R58 to R61, R59 to R62, R60 to R63, R61 to R64, R62 to R65, R63 to R66, R64 to R67, R65 to R68, R66 to R69, R67 to R70, R68 to R71, R69 to R72, R70 to R73, R71 to R74, R72 to R75, R73 to R76, R74 to R77, R75 to R78, R76 to R79, R77 to R80, R78 to R81, R79 to R82, U9 to U10, U10 to U11, U11 to U12, U12 to U13, U13 to U14, U14 to U15, U15 to U16, U16 to U17, U5 to U6, U6 to U7, U7 to U8
Connections:
- C3 pad 1: /CM4/I2C GPIO1/+3.3V_IN -> +12V
- C4 pad 1: /CM4/I2C GPIO1/+3.3V_IN -> +12V
- CM1 pad 45: /CM4/~{INT_CM4} -> /CM4/~{PANIC_CM4}
- CM1 pad 47: /CM4/CM4 Hirose connectors/GPIO23 -> /CM4/~{INT_CM4}
- R3 pad 1: /CM4/I2C GPIO1/~{I2C_RESET} -> /CM4/~{I2C_RESET_1_2}
- R3 pad 2: /CM4/I2C GPIO1/+3.3V_IN -> +12V
- R34 pad 1: +12V -> /PRSNT_BOARD_X1_1
- R34 pad 2: /PRSNT_BOARD_X1_1 -> +12V
- R35 pad 1: +12V -> /PRSNT_BOARD_X8_1
- R35 pad 2: /PRSNT_BOARD_X8_1 -> +12V
- R36 pad 1: +12V -> /PRSNT_BOARD_X4_1
- R36 pad 2: /PRSNT_BOARD_X4_1 -> +12V
- U2 pad 19: /CM4/I2C GPIO1/I2C_SCL -> /CM4/I2C_SCL
- U2 pad 20: /CM4/I2C GPIO1/I2C_SDA -> /CM4/I2C_SDA
- U2 pad 21: /CM4/I2C GPIO1/+3.3V_IN -> +12V
- U2 pad 22: /CM4/I2C GPIO1/~{I2C_RESET} -> /CM4/~{I2C_RESET_1_2}

Commit message: layout experiments
Parts:
- moved R77 90.6 mm to (53.7, 93.8), turned to 90 degrees
- moved R79 89.7 mm to (51.7, 93.8), turned to 90 degrees
- moved R76 89.5 mm to (54.8, 93.8), turned to 90 degrees
- moved R82 88.8 mm to (48.5, 93.8), turned to 90 degrees
- moved R72 88.1 mm to (58.9, 93.8), turned to 90 degrees
- moved R75 87.8 mm to (55.8, 93.8), turned to 90 degrees
- moved R78 86.3 mm to (52.7, 93.8), turned to 90 degrees
- moved R71 85.6 mm to (59.9, 93.8), turned to 90 degrees
- moved R74 84.3 mm to (56.8, 93.8), turned to 90 degrees
- moved R73 81.7 mm to (57.9, 93.8), turned to 90 degrees
- moved C74 79.9 mm to (54.4, 81.2)
- moved C71 77.2 mm to (58.4, 81.2)
- moved C72 76.5 mm to (43.2, 81.2), turned to 90 degrees
- moved C78 74.9 mm to (57.4, 81.2), turned to 90 degrees
- moved C76 73.7 mm to (41.2, 81.2), turned to 90 degrees
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Routing:
- added copper zone on B.Cu, net GND
- added copper zone on F.Cu, net GND
- added copper zone on In1.Cu, net GND
- added copper zone on In2.Cu, net GND
- removed copper zone on B.Cu, net (none)
- removed copper zone on F.Cu, net (none)
