File: cm4.kicad_sch (KiCad schematic)
At the start: 54 parts, among them Q1 MMBT2222AM3T5G, U3 SN74LVC1G04DRY, U4 SN74LVC1G07DRY, U5 PCA9641BSHP

Commit message: schematic sheet renames
Other:
- sheet Sensors: file cm4sensors.kicad_sch -> tempsensors.kicad_sch
Changed lines of the file:
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@@
       (effects (font (size 3 3) bold italic) (justify left bottom))
     )
-    (property "Sheet file" "cm4sensors.kicad_sch" (id 1) (at 534.67 174.9984 0)
+    (property "Sheet file" "tempsensors.kicad_sch" (id 1) (at 534.67 174.9984 0)
       (effects (font (size 1.27 1.27)) (justify left top) hide)
     )

Commit message: work on control logic
Parts:
- added C7: 10uF, Capacitor_SMD:C_0402_1005Metric, symbol Device:C_Small
- added C8: 0.1uF, Capacitor_SMD:C_0402_1005Metric, symbol Device:C_Small
- added R13, R14: 1k, Resistor_SMD:R_0402_1005Metric, symbol Device:R_Small
- added R37: 10k, Resistor_SMD:R_0402_1005Metric, symbol Device:R_Small
- added U5: SN74HCS244, Buffer_SMD_TI:RKS0020A, symbol Buffer_SMD_TI:SN74HCS244
- renumbered C8 to C10, C7 to C9, R13 to R15, R14 to R16, R15 to R17, R16 to R18, R17 to R19, R18 to R20, R19 to R21, R20 to R22, R21 to R23, R25 to R24, R26 to R25, R27 to R26, R28 to R27, R29 to R28, R30 to R29, R31 to R30, R32 to R31, R33 to R32, R34 to R33, R22 to R34, R23 to R35, R24 to R36, U5 to U6
Connections:
- net +3.3V_CONTROL: now also R34.2, R35.2, R36.2, C7.1, C8.1, R13.2, R14.2, R37.2, U5.20 (VCC); no longer R34.1, R35.1, R36.1
- net GND: now also C7.2, C8.2
- net ~{I2C_RESET_1_1}: now also U5.18 (1Y1)
- net ~{I2C_RESET_1_2}: now also U5.16 (1Y2)
- net ~{I2C_RESET_1}: now also U5.2 (1A1), U5.4 (1A2)
- net ~{INT_CM4}: now also R37.1, U5.11 (2A1), U5.13 (2A2)
- net ~{PANIC}: now also U5.9 (2Y1)
- net ~{PRSNT_BOARD_X1_1}: now also R34.1; no longer R34.2
- net ~{PRSNT_BOARD_X4_1}: now also R35.1; no longer R35.2
- net ~{PRSNT_BOARD_X8_1}: now also R36.1; no longer R36.2
- new net: R13.1, U5.1 (1~{OE})
- new net: R14.1, U5.19 (2~{OE})
- new net ePAD: U5.10 (GND), U5.15 (2A3), U5.17 (2A4), U5.21 (ePAD), U5.6 (1A3), U5.8 (1A4)
- new net ~{PANIC_CM4}: U5.7 (2Y2)
- no-connect marks 25 -> 28
Other:
- note added: "Listening to local ~{INT}"
- note added: "~{INT} trigger for CM4"
- moved on the sheet: R34, R35, R36

Commit message: work on control logic
Connections:
- net ePAD is gone; now on net GND: U5.10 (GND), U5.15 (2A3), U5.17 (2A4), U5.21 (ePAD), U5.6 (1A3), U5.8 (1A4)
- net ~{I2C_RESET_1_1}: no longer R28.1
- net ~{I2C_RESET_1}: now also R28.1
Other:
- note added: "Not clear this is needed."
Changed lines of the file:
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@@
     (effects (font (size 5 5) (thickness 1) bold italic) (justify left bottom))
+  )
+  (text "Not clear this is needed." (at 774.7 381 0)
+    (effects (font (size 1.27 1.27)) (justify left bottom))
   )
   (text "Output" (at 632.46 229.87 0)
@@
     (effects (font (size 1.27 1.27)) (justify right bottom))
   )
-  (label "~{I2C_RESET_1_1}" (at 755.65 381 180)
+  (label "~{I2C_RESET_CM4}" (at 755.65 381 180)
     (effects (font (size 1.27 1.27)) (justify right bottom))
   )
@@
       (effects (font (size 1.27 1.27)) hide)
     )
+    (pin "1")
+  )
+  (symbol (lib_id "power:GND") (at 574.04 407.67 0) (unit 1)
+    (in_bom yes) (on_board yes) (fields_autoplaced)
+    (property "Reference" "#PWR?" (id 0) (at 574.04 414.02 0)
+      (effects (font (size 1.27 1.27)) hide)
+    )
+    (property "Value" "GND" (id 1) (at 574.04 412.75 0))
+    (property "Footprint" "" (id 2) (at 574.04 407.67 0)
+      (effects (font (size 1.27 1.27)) hide)
+    )
+    (property "Datasheet" "" (id 3) (at 574.04 407.67 0)
+      (effects (font (size 1.27 1.27)) hide)
+    )

Commit message: refresh
Parts:
- removed C6: 0.1uF, Capacitor_SMD:C_0402_1005Metric, symbol Device:C_Small
- removed U4: SN74LVC1G07DRY, Buffer_SMD_TI:PSON50P145X100X60-6N-DRY0006A, symbol Buffer_SMD_TI:SN74LVC1G07DRY
Connections:
- net GND: no longer U5.17 (2A4)
- net ~{PWR_LED}: now also U5.17 (2A4)
- net ~{PWR_LED_BUFFERED}: now reaches D2.1 (K), TP3.1
- net ~{PWR_LED_BUFFERED}: now also U5.3 (2Y4)
- no-connect marks 28 -> 27
Other:
- moved on the sheet: D3, D4, D5, D6, R6, R7, R8, R9, TP3, TP4, TP5, TP6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

Commit message: merging changes for face plate conn
Parts:
- removed D1: LED Blue, LED_SMD_LiteOn:LED_0603_1608Metric_blue, symbol LED_SMD_LiteOn:LED Blue
- removed D2: LED Red, LED_SMD_LiteOn:LED_0603_1608Metric_red, symbol LED_SMD_LiteOn:LED Red
- removed D3, D5: LED Green, LED_SMD_LiteOn:LED_0603_1608Metric_green, symbol LED_SMD_LiteOn:LED Green
- removed D4: LED Yellow, LED_SMD_LiteOn:LED_0603_1608Metric_yellow, symbol LED_SMD_LiteOn:LED Yellow
- removed D6: LED Orange, LED_SMD_LiteOn:LED_0603_1608Metric_orange, symbol LED_SMD_LiteOn:LED Orange
- removed LED1: APHB1608CGKSEKC_KNB, LED_SMD_Kingbright:APHB1608CGKSEKC, symbol LED_SMD_Kingbright:APHB1608CGKSEKC_KNB
Connections:
- net +3.3V_CONTROL: no longer R19.2
- net CM4_+3.3V: no longer R5.2, R6.2, R7.1, R8.1, R9.1
- net ~{EthLED1}: now also R7.1
- net ~{EthLED2}: now also R8.1
- net ~{EthLED3}: now also R9.1
- net ~{PI_Activity}: now also R6.2
- net ~{PWR_LED_BUFFERED}: now also R5.2
- net ~{LED_EthLED2_CONN}: now reaches R8.2
- net ~{LED_EthLED3_CONN}: now reaches R9.2
- net ~{M.2_LED_CONN}: now reaches R4.1
- net ~{LED_PI_Activity_CONN}: now reaches R6.1
- net LED_I2C_PING_1_CONN: now reaches R19.1
- net ~{LED_PWR_LED_BUFFERED_CONN}: now reaches R5.1
- net at Q1.3 (C), R17.2, TP9.1: now also R19.2
- net LED_+3.3V_ON_CONN: now reaches R18.1
- net ~{LED_EthLED1_CONN}: now reaches R7.2
Other:
- sheet USB 2.0 MUX ports: added LED_USB_OTG; removed none
- moved on the sheet: R18, R19, R5, R6, R7, R8, R9

Commit message: refresh
Parts:
- added J?: PicoBlade_1x12_533981371_SMT, Connector_PicoBlade_Molex:MOLEX_533981271, symbol Connector_PicoBlade_Molex:PicoBlade_1x12_533981371_SMT
Connections:
- net +3.3V_CONTROL: now also J?.9 (Pin_9)
- net CM4_+3.3V: now also J?.11 (Pin_11)
- net GND: now also J?.12 (Pin_12), J?.S (SHIELD)
- net LED_+3.3V_ON_CONN: now also J?.7 (Pin_7)
- net LED_I2C_PING_1_CONN: now also J?.8 (Pin_8)
- net LED_USB_OTG_CONN: now also J?.10 (Pin_10)
- net ~{LED_EthLED1_CONN}: now also J?.4 (Pin_4)
- net ~{LED_EthLED2_CONN}: now also J?.5 (Pin_5)
- net ~{LED_EthLED3_CONN}: now also J?.6 (Pin_6)
- net ~{LED_PI_Activity_CONN}: now also J?.3 (Pin_3)
- net ~{LED_PWR_LED_BUFFERED_CONN}: now also J?.2 (Pin_2)
- net ~{M.2_LED_CONN}: now also J?.1 (Pin_1)
Changed lines of the file:
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@@
   (junction (at 720.09 429.26) (diameter 0) (color 0 0 0 0)
+  )
+  (junction (at 179.07 426.72) (diameter 0) (color 0 0 0 0)
   )
   (junction (at 695.96 220.98) (diameter 0) (color 0 0 0 0)
@@
     (stroke (width 0) (type solid) (color 0 0 0 0))
   )
+  (wire (pts (xy 133.35 401.32) (xy 179.07 401.32))
+    (stroke (width 0) (type default) (color 0 0 0 0))
+  )
   (wire (pts (xy 238.76 509.27) (xy 267.97 509.27))
     (stroke (width 0) (type solid) (color 0 0 0 0))
@@
     (stroke (width 0) (type solid) (color 0 0 0 0))
   )
+  (wire (pts (xy 179.07 424.18) (xy 179.07 426.72))
+    (stroke (width 0) (type default) (color 0 0 0 0))
+  )
   (wire (pts (xy 148.59 537.21) (xy 168.91 537.21))
     (stroke (width 0) (type solid) (color 0 0 0 0))
@@
     (stroke (width 0) (type default) (color 0 0 0 0))
   )
+  (wire (pts (xy 133.35 398.78) (xy 179.07 398.78))
+    (stroke (width 0) (type default) (color 0 0 0 0))
+  )
   (wire (pts (xy 720.09 381) (xy 720.09 388.62))
     (stroke (width 0) (type default) (color 0 0 0 0))
@@
     (stroke (width 0) (type solid) (color 0 0 0 0))
   )
+  (wire (pts (xy 133.35 419.1) (xy 179.07 419.1))
+    (stroke (width 0) (type default) (color 0 0 0 0))
+  )
   (wire (pts (xy 546.1 539.75) (xy 566.42 539.75))
     (stroke (width 0) (type default) (color 0 0 0 0))
   )
+  (wire (pts (xy 133.35 414.02) (xy 179.07 414.02))
+    (stroke (width 0) (type default) (color 0 0 0 0))
+  )
   (wire (pts (xy 300.99 509.27) (xy 325.12 509.27))
     (stroke (width 0) (type solid) (color 0 0 0 0))
@@
   (wire (pts (xy 78.74 195.58) (xy 114.3 195.58))
     (stroke (width 0) (type solid) (color 0 0 0 0))
+  )
+  (wire (pts (xy 133.35 421.64) (xy 179.07 421.64))
+    (stroke (width 0) (type default) (color 0 0 0 0))
   )
   (wire (pts (xy 720.09 431.8) (xy 720.09 439.42))
@@
     (stroke (width 0) (type default) (color 0 0 0 0))
   )
+  (wire (pts (xy 133.35 403.86) (xy 179.07 403.86))
+    (stroke (width 0) (type default) (color 0 0 0 0))
+  )
   (wire (pts (xy 78.74 179.07) (xy 114.3 179.07))
     (stroke (width 0) (type solid) (color 0 0 0 0))
@@
   )
   (wire (pts (xy 610.87 208.28) (xy 562.61 208.28))
+    (stroke (width 0) (type default) (color 0 0 0 0))
+  )
+  (wire (pts (xy 133.35 426.72) (xy 179.07 426.72))
     (stroke (width 0) (type default) (color 0 0 0 0))
   )
@@
     (stroke (width 0) (type solid) (color 0 0 0 0))
   )
+  (wire (pts (xy 133.35 411.48) (xy 179.07 411.48))
+    (stroke (width 0) (type default) (color 0 0 0 0))
+  )
   (wire (pts (xy 549.91 350.52) (xy 549.91 347.98))
     (stroke (width 0) (type default) (color 0 0 0 0))
@@
     (stroke (width 0) (type default) (color 0 0 0 0))
   )
+  (wire (pts (xy 179.07 426.72) (xy 179.07 433.07))
+    (stroke (width 0) (type default) (color 0 0 0 0))
+  )
   (wire (pts (xy 300.99 266.7) (xy 283.21 266.7))
     (stroke (width 0) (type solid) (color 0 0 0 0))
@@
     (stroke (width 0) (type default) (color 0 0 0 0))
   )
+  (wire (pts (xy 133.35 424.18) (xy 179.07 424.18))
+    (stroke (width 0) (type default) (color 0 0 0 0))
+  )
   (wire (pts (xy 754.38 177.8) (xy 772.16 177.8))
     (stroke (width 0) (type default) (color 0 0 0 0))
@@
     (stroke (width 0) (type default) (color 0 0 0 0))
   )
+  (wire (pts (xy 133.35 406.4) (xy 179.07 406.4))
+    (stroke (width 0) (type default) (color 0 0 0 0))
+  )
   (wire (pts (xy 300.99 311.15) (xy 283.21 311.15))
     (stroke (width 0) (type solid) (color 0 0 0 0))
   )
+  (wire (pts (xy 133.35 396.24) (xy 179.07 396.24))
+    (stroke (width 0) (type default) (color 0 0 0 0))
+  )
   (wire (pts (xy 191.77 179.07) (xy 156.21 179.07))
     (stroke (width 0) (type solid) (color 0 0 0 0))
@@
     (stroke (width 0) (type solid) (color 0 0 0 0))
   )
+  (wire (pts (xy 133.35 408.94) (xy 179.07 408.94))
+    (stroke (width 0) (type default) (color 0 0 0 0))
+  )
   (wire (pts (xy 492.76 229.87) (xy 534.67 229.87))
     (stroke (width 0) (type default) (color 0 0 0 0))
@@
   )
   (wire (pts (xy 552.45 382.27) (xy 576.58 382.27))
+    (stroke (width 0) (type default) (color 0 0 0 0))
+  )
+  (wire (pts (xy 133.35 416.56) (xy 179.07 416.56))
     (stroke (width 0) (type default) (color 0 0 0 0))
   )
@@
     (effects (font (size 1.27 1.27)) (justify right bottom))
   )
+  (label "~{LED_EthLED3_CONN}" (at 179.07 408.94 180)
+    (effects (font (size 1.27 1.27)) (justify right bottom))
+  )
   (label "~{INT_BACKPLANE}" (at 755.65 396.24 180)
     (effects (font (size 1.27 1.27)) (justify right bottom))
@@
     (effects (font (size 1.27 1.27)) (justify right bottom))
   )
+  (label "~{LED_PWR_LED_BUFFERED_CONN}" (at 179.07 398.78 180)
+    (effects (font (size 1.27 1.27)) (justify right bottom))
+  )
   (label "HDMICK+" (at 283.21 330.2 0)
     (effects (font (size 1.27 1.27)) (justify left bottom))
@@
     (effects (font (size 1.27 1.27)) (justify right bottom))
   )
+  (label "~{LED_EthLED2_CONN}" (at 179.07 406.4 180)
+    (effects (font (size 1.27 1.27)) (justify right bottom))
+  )
   (label "HDMIHP" (at 283.21 339.09 0)
     (effects (font (size 1.27 1.27)) (justify left bottom))
@@
     (effects (font (size 1.27 1.27)) (justify left bottom))
   )
+  (label "LED_+3.3V" (at 179.07 421.64 180)
+    (effects (font (size 1.27 1.27)) (justify right bottom))
+  )
   (label "HDMIHP" (at 191.77 335.28 180)
     (effects (font (size 1.27 1.27)) (justify right bottom))
@@
     (effects (font (size 1.27 1.27)) (justify right bottom))
   )
+  (label "LED_I2C_PING_1_CONN" (at 179.07 414.02 180)
+    (effects (font (size 1.27 1.27)) (justify right bottom))
+  )
   (label "SD_PWR_ON" (at 284.48 194.31 0)
     (effects (font (size 1.27 1.27)) (justify left bottom))
@@
     (effects (font (size 1.27 1.27)) (justify right bottom))
   )
+  (label "~{LED_PI_Activity_CONN}" (at 179.07 401.32 180)
+    (effects (font (size 1.27 1.27)) (justify right bottom))
+  )
   (label "CM4_I2C_SDA" (at 755.65 373.38 180)
     (effects (font (size 1.27 1.27)) (justify right bottom))
@@
     (effects (font (size 1.27 1.27)) (justify right bottom))
   )
+  (label "LED_USB_OTG_CONN" (at 179.07 419.1 180)
+    (effects (font (size 1.27 1.27)) (justify right bottom))
+  )
   (label "~{I2C_RESET_1_2}" (at 755.65 419.1 180)
     (effects (font (size 1.27 1.27)) (justify right bottom))
@@
     (effects (font (size 1.27 1.27)) (justify right bottom))
   )
+  (label "LED_+3.3V_CONTROL_CONN" (at 179.07 416.56 180)
+    (effects (font (size 1.27 1.27)) (justify right bottom))
+  )
+  (label "~{LED_EthLED1_CONN}" (at 179.07 403.86 180)
+    (effects (font (size 1.27 1.27)) (justify right bottom))
+  )
   (label "I2C_SCL" (at 494.03 168.91 0)
     (effects (font (size 1.27 1.27)) (justify left bottom))
@@
     (effects (font (size 1.27 1.27)) (justify left bottom))
   )
+  (label "~{M.2_LED_CONN}" (at 179.07 396.24 180)
+    (effects (font (size 1.27 1.27)) (justify right bottom))
+  )
   (label "HDMID0+" (at 191.77 307.34 180)
     (effects (font (size 1.27 1.27)) (justify right bottom))
@@
   (label "~{INT_CM4}" (at 662.94 198.12 0)
     (effects (font (size 1.27 1.27)) (justify left bottom))
+  )
+  (label "LED_+3.3V_ON_CONN" (at 179.07 411.48 180)
+    (effects (font (size 1.27 1.27)) (justify right bottom))
   )
   (label "~{EthLED1}" (at 78.74 179.07 0)
@@
     (pin "1")
     (pin "2")
+  )
+  (symbol (lib_id "Connector_PicoBlade_Molex:PicoBlade_1x12_533981371_SMT") (at 128.27 403.86 0) (mirror y) (unit 1)
+    (in_bom yes) (on_board yes) (fields_autoplaced)
+    (property "Reference" "J?" (id 0) (at 128.27 389.89 0))
+    (property "Value" "PicoBlade_1x12_533981371_SMT" (id 1) (at 128.27 392.43 0))
+    (property "Footprint" "Connector_PicoBlade_Molex:MOLEX_533981271" (id 2) (at 128.27 438.15 0)
+      (effects (font (size 1.27 1.27)) hide)
+    )
+    (property "Datasheet" "~" (id 3) (at 128.27 403.86 0)
+      (effects (font (size 1.27 1.27)) hide)
+    )
+    (property "Manufacturer" "Molex" (id 4) (at 128.27 433.07 0)
+      (effects (font (size 1.27 1.27)) hide)
+    )
+    (property "MPN" "533981271" (id 5) (at 128.27 435.61 0)
+      (effects (font (size 1.27 1.27)) hide)
+    )
+    (pin "10")
+    (pin "11")
+    (pin "12")
+    (pin "9")
+    (pin "S")
+    (pin "1")
+    (pin "2")
+    (pin "3")
+    (pin "4")
+    (pin "5")
+    (pin "6")
+    (pin "7")
+    (pin "8")
   )
   (symbol (lib_id "Device:C_Small") (at 671.83 133.35 0) (unit 1)
@@
     (pin "2")
   )
+  (symbol (lib_id "power:GND") (at 179.07 433.07 0) (unit 1)
+    (in_bom yes) (on_board yes) (fields_autoplaced)
+    (property "Reference" "#PWR?" (id 0) (at 179.07 439.42 0)
+      (effects (font (size 1.27 1.27)) hide)
+    )
+    (property "Value" "GND" (id 1) (at 179.07 438.15 0))
+    (property "Footprint" "" (id 2) (at 179.07 433.07 0)
+      (effects (font (size 1.27 1.27)) hide)
+    )
+    (property "Datasheet" "" (id 3) (at 179.07 433.07 0)
+      (effects (font (size 1.27 1.27)) hide)
+    )
+    (pin "1")
+  )
   (symbol (lib_id "Device:R_Small") (at 436.88 534.67 270) (mirror x) (unit 1)

Commit message: connecterized faceplate, refreshed schematic
Parts:
- gave numbers to parts that had none: 1
- renumbered C7 to C6, C8 to C7, C9 to C8, C10 to C9, U5 to U4, U6 to U5
Changed lines of the file:
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@@
   (symbol (lib_id "Device:C_Small") (at 549.91 345.44 0) (unit 1)
     (in_bom yes) (on_board yes)
-    (property "Reference" "C8" (id 0) (at 551.815 344.17 0)
+    (property "Reference" "C7" (id 0) (at 551.815 344.17 0)
       (effects (font (size 1.27 1.27)) (justify left))
     )
@@
   (symbol (lib_id "Connector_PicoBlade_Molex:PicoBlade_1x12_533981371_SMT") (at 128.27 403.86 0) (mirror y) (unit 1)
     (in_bom yes) (on_board yes) (fields_autoplaced)
-    (property "Reference" "J?" (id 0) (at 128.27 389.89 0))
+    (property "Reference" "J2" (id 0) (at 128.27 389.89 0))
     (property "Value" "PicoBlade_1x12_533981371_SMT" (id 1) (at 128.27 392.43 0))
     (property "Footprint" "Connector_PicoBlade_Molex:MOLEX_533981271" (id 2) (at 128.27 438.15 0)
@@
   (symbol (lib_id "Device:C_Small") (at 671.83 133.35 0) (unit 1)
     (in_bom yes) (on_board yes)
-    (property "Reference" "C9" (id 0) (at 673.735 132.08 0)
+    (property "Reference" "C8" (id 0) (at 673.735 132.08 0)
       (effects (font (size 1.27 1.27)) (justify left))
     )
@@
   (symbol (lib_id "Interface_I2C_NXP:PCA9641BSHP") (at 693.42 157.48 0) (unit 1)
     (in_bom yes) (on_board yes) (fields_autoplaced)
-    (property "Reference" "U6" (id 0) (at 740.41 148.59 0))
+    (property "Reference" "U5" (id 0) (at 740.41 148.59 0))
     (property "Value" "PCA9641BSHP" (id 1) (at 745.49 226.06 0))
     (property "Footprint" "Interface_I2C_NXP:SOT758-1_HVQFN-16_3x3mm_P0.5mm_EP1.75x1.75mm_NXP" (id 2) (at 740.41 237.49 0)
@@
   (symbol (lib_id "power:GND") (at 519.43 245.11 0) (unit 1)
     (in_bom yes) (on_board yes) (fields_autoplaced)
-    (property "Reference" "#PWR09" (id 0) (at 519.43 251.46 0)
+    (property "Reference" "#PWR08" (id 0) (at 519.43 251.46 0)
       (effects (font (size 1.27 1.27)) hide)
     )
@@
   (symbol (lib_id "power:GND") (at 695.96 236.22 0) (unit 1)
     (in_bom yes) (on_board yes) (fields_autoplaced)
-    (property "Reference" "#PWR015" (id 0) (at 695.96 242.57 0)
+    (property "Reference" "#PWR014" (id 0) (at 695.96 242.57 0)
       (effects (font (size 1.27 1.27)) hide)
     )
@@
   (symbol (lib_id "Device:C_Small") (at 684.53 133.35 0) (unit 1)
     (in_bom yes) (on_board yes)
-    (property "Reference" "C10" (id 0) (at 686.435 132.08 0)
+    (property "Reference" "C9" (id 0) (at 686.435 132.08 0)
       (effects (font (size 1.27 1.27)) (justify left))
     )
@@
   (symbol (lib_id "power:GND") (at 574.04 407.67 0) (unit 1)
     (in_bom yes) (on_board yes) (fields_autoplaced)
-    (property "Reference" "#PWR?" (id 0) (at 574.04 414.02 0)
+    (property "Reference" "#PWR010" (id 0) (at 574.04 414.02 0)
       (effects (font (size 1.27 1.27)) hide)
     )
@@
   (symbol (lib_id "Buffer_SMD_TI:SN74HCS244") (at 576.58 359.41 0) (unit 1)
     (in_bom yes) (on_board yes)
-    (property "Reference" "U5" (id 0) (at 580.39 355.6 0))
+    (property "Reference" "U4" (id 0) (at 580.39 355.6 0))
     (property "Value" "SN74HCS244" (id 1) (at 601.98 398.78 0)
       (effects (font (size 1.27 1.27)) (justify right))
@@
   (symbol (lib_id "power:GND") (at 684.53 139.7 0) (unit 1)
     (in_bom yes) (on_board yes) (fields_autoplaced)
-    (property "Reference" "#PWR014" (id 0) (at 684.53 146.05 0)
+    (property "Reference" "#PWR013" (id 0) (at 684.53 146.05 0)
       (effects (font (size 1.27 1.27)) hide)
     )
@@
   (symbol (lib_id "power:GND") (at 549.91 351.79 0) (unit 1)
     (in_bom yes) (on_board yes) (fields_autoplaced)
-    (property "Reference" "#PWR010" (id 0) (at 549.91 358.14 0)
+    (property "Reference" "#PWR09" (id 0) (at 549.91 358.14 0)
       (effects (font (size 1.27 1.27)) hide)
     )
@@
   (symbol (lib_id "Device:C_Small") (at 539.75 345.44 0) (unit 1)
     (in_bom yes) (on_board yes)
-    (property "Reference" "C7" (id 0) (at 541.655 344.17 0)
+    (property "Reference" "C6" (id 0) (at 541.655 344.17 0)
       (effects (font (size 1.27 1.27)) (justify left))
     )
@@
   (symbol (lib_id "power:GND") (at 179.07 433.07 0) (unit 1)
     (in_bom yes) (on_board yes) (fields_autoplaced)
-    (property "Reference" "#PWR?" (id 0) (at 179.07 439.42 0)
+    (property "Reference" "#PWR06" (id 0) (at 179.07 439.42 0)
       (effects (font (size 1.27 1.27)) hide)
     )
@@
   (symbol (lib_id "power:GND") (at 273.05 515.62 0) (unit 1)
     (in_bom yes) (on_board yes)
-    (property "Reference" "#PWR06" (id 0) (at 273.05 521.97 0)
-      (effects (font (size 1.27 1.27)) hide)
-    )
+    (property "Reference" "#PWR07" (id 0) (at 273.05 521.97 0)
+      (effects (font (size 1.27 1.27)) hide)
+    )

Commit message: placed hdmi conn
Other:
- note added: "Indicators - I2C Diagnostic"
- note removed: "Indicators - I2C"
