File: cm4m2mkey.kicad_sch (KiCad schematic)
At the start: 26 parts, among them J8 1-2199119-6

Commit message: board refresh
Parts:
- renumbered C68 to C66, C69 to C67, C70 to C68, C71 to C69, C72 to C70, C73 to C71, C74 to C72, C75 to C73, C76 to C74, C77 to C75, C78 to C76, R61 to R64, R62 to R65, R63 to R66, R64 to R67, R65 to R68, R66 to R69, R67 to R70, R68 to R71, R69 to R72, R70 to R73, R71 to R74, R72 to R75, R73 to R76, R74 to R77
Changed lines of the file:
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@@
   (symbol (lib_id "Device:R_Small") (at 81.28 118.11 90) (unit 1)
     (in_bom yes) (on_board yes)
-    (property "Reference" "R61" (id 0) (at 74.93 116.84 90)
+    (property "Reference" "R64" (id 0) (at 74.93 116.84 90)
       (effects (font (size 1 1)) (justify right))
     )
@@
   (symbol (lib_id "Device:R_Small") (at 99.06 77.47 90) (unit 1)
     (in_bom yes) (on_board yes)
-    (property "Reference" "R68" (id 0) (at 92.71 76.2 90)
+    (property "Reference" "R71" (id 0) (at 92.71 76.2 90)
       (effects (font (size 1 1)) (justify right))
     )
@@
   (symbol (lib_id "Device:C_Small") (at 147.32 54.61 90) (unit 1)
     (in_bom yes) (on_board yes)
-    (property "Reference" "C70" (id 0) (at 146.05 53.34 90)
+    (property "Reference" "C68" (id 0) (at 146.05 53.34 90)
       (effects (font (size 1 1)) (justify left))
     )
@@
   (symbol (lib_id "Device:R_Small") (at 99.06 82.55 90) (unit 1)
     (in_bom yes) (on_board yes)
-    (property "Reference" "R69" (id 0) (at 92.71 81.28 90)
+    (property "Reference" "R72" (id 0) (at 92.71 81.28 90)
       (effects (font (size 1 1)) (justify right))
     )
@@
   (symbol (lib_id "Device:C_Small") (at 147.32 167.64 90) (unit 1)
     (in_bom yes) (on_board yes)
-    (property "Reference" "C78" (id 0) (at 146.05 166.37 90)
+    (property "Reference" "C76" (id 0) (at 146.05 166.37 90)
       (effects (font (size 1 1)) (justify left))
     )
@@
   (symbol (lib_id "Device:R_Small") (at 99.06 74.93 90) (unit 1)
     (in_bom yes) (on_board yes)
-    (property "Reference" "R67" (id 0) (at 92.71 73.66 90)
+    (property "Reference" "R70" (id 0) (at 92.71 73.66 90)
       (effects (font (size 1 1)) (justify right))
     )
@@
   (symbol (lib_id "Device:R_Small") (at 99.06 59.69 90) (unit 1)
     (in_bom yes) (on_board yes)
-    (property "Reference" "R63" (id 0) (at 93.345 58.801 90)
+    (property "Reference" "R66" (id 0) (at 93.345 58.801 90)
       (effects (font (size 1 1)) (justify right))
     )
@@
   (symbol (lib_id "Device:R_Small") (at 99.06 67.31 90) (unit 1)
     (in_bom yes) (on_board yes)
-    (property "Reference" "R65" (id 0) (at 92.71 66.04 90)
+    (property "Reference" "R68" (id 0) (at 92.71 66.04 90)
       (effects (font (size 1 1)) (justify right))
     )
@@
   (symbol (lib_id "Device:C_Small") (at 147.32 152.4 90) (unit 1)
     (in_bom yes) (on_board yes)
-    (property "Reference" "C74" (id 0) (at 146.05 151.13 90)
+    (property "Reference" "C72" (id 0) (at 146.05 151.13 90)
       (effects (font (size 1 1)) (justify left))
     )
@@
   (symbol (lib_id "Device:C_Small") (at 147.32 144.78 90) (unit 1)
     (in_bom yes) (on_board yes)
-    (property "Reference" "C72" (id 0) (at 146.05 143.51 90)
+    (property "Reference" "C70" (id 0) (at 146.05 143.51 90)
       (effects (font (size 1 1)) (justify left))
     )
@@
   (symbol (lib_id "Device:C_Small") (at 147.32 140.97 90) (unit 1)
     (in_bom yes) (on_board yes)
-    (property "Reference" "C71" (id 0) (at 146.05 139.7 90)
+    (property "Reference" "C69" (id 0) (at 146.05 139.7 90)
       (effects (font (size 1 1)) (justify left))
     )
@@
   (symbol (lib_id "Device:R_Small") (at 99.06 97.79 90) (unit 1)
     (in_bom yes) (on_board yes)
-    (property "Reference" "R73" (id 0) (at 92.71 96.52 90)
+    (property "Reference" "R76" (id 0) (at 92.71 96.52 90)
       (effects (font (size 1 1)) (justify right))
     )
@@
   (symbol (lib_id "Device:C_Small") (at 147.32 148.59 90) (unit 1)
     (in_bom yes) (on_board yes)
-    (property "Reference" "C73" (id 0) (at 146.05 147.32 90)
+    (property "Reference" "C71" (id 0) (at 146.05 147.32 90)
       (effects (font (size 1 1)) (justify left))
     )
@@
   (symbol (lib_id "Device:C_Small") (at 147.32 46.99 90) (unit 1)
     (in_bom yes) (on_board yes)
-    (property "Reference" "C68" (id 0) (at 146.05 45.72 90)
+    (property "Reference" "C66" (id 0) (at 146.05 45.72 90)
       (effects (font (size 1 1)) (justify left))
     )
@@
   (symbol (lib_id "power:GND") (at 90.17 153.67 0) (unit 1)
     (in_bom yes) (on_board yes)
-    (property "Reference" "#PWR057" (id 0) (at 90.17 160.02 0)
+    (property "Reference" "#PWR055" (id 0) (at 90.17 160.02 0)
       (effects (font (size 1.27 1.27)) hide)
     )
@@
   (symbol (lib_id "power:GND") (at 154.94 170.18 0) (unit 1)
     (in_bom yes) (on_board yes)
-    (property "Reference" "#PWR059" (id 0) (at 154.94 176.53 0)
+    (property "Reference" "#PWR057" (id 0) (at 154.94 176.53 0)
       (effects (font (size 1.27 1.27)) hide)
     )
@@
   (symbol (lib_id "Device:R_Small") (at 99.06 69.85 90) (unit 1)
     (in_bom yes) (on_board yes)
-    (property "Reference" "R66" (id 0) (at 92.71 68.58 90)
+    (property "Reference" "R69" (id 0) (at 92.71 68.58 90)
       (effects (font (size 1 1)) (justify right))
     )
@@
   (symbol (lib_id "Device:C_Small") (at 147.32 163.83 90) (unit 1)
     (in_bom yes) (on_board yes)
-    (property "Reference" "C77" (id 0) (at 146.05 162.56 90)
+    (property "Reference" "C75" (id 0) (at 146.05 162.56 90)
       (effects (font (size 1 1)) (justify left))
     )
@@
   (symbol (lib_id "Device:C_Small") (at 147.32 156.21 90) (unit 1)
     (in_bom yes) (on_board yes)
-    (property "Reference" "C75" (id 0) (at 146.05 154.94 90)
+    (property "Reference" "C73" (id 0) (at 146.05 154.94 90)
       (effects (font (size 1 1)) (justify left))
     )
@@
   (symbol (lib_id "power:GND") (at 154.94 57.15 0) (unit 1)
     (in_bom yes) (on_board yes)
-    (property "Reference" "#PWR058" (id 0) (at 154.94 63.5 0)
+    (property "Reference" "#PWR056" (id 0) (at 154.94 63.5 0)
       (effects (font (size 1.27 1.27)) hide)
     )
@@
   (symbol (lib_id "Device:R_Small") (at 99.06 90.17 90) (unit 1)
     (in_bom yes) (on_board yes)
-    (property "Reference" "R71" (id 0) (at 92.71 88.9 90)
+    (property "Reference" "R74" (id 0) (at 92.71 88.9 90)
       (effects (font (size 1 1)) (justify right))
     )
@@
   (symbol (lib_id "Device:R_Small") (at 99.06 62.23 90) (unit 1)
     (in_bom yes) (on_board yes)
-    (property "Reference" "R64" (id 0) (at 92.71 60.96 90)
+    (property "Reference" "R67" (id 0) (at 92.71 60.96 90)
       (effects (font (size 1 1)) (justify right))
     )
@@
   (symbol (lib_id "Device:C_Small") (at 147.32 50.8 90) (unit 1)
     (in_bom yes) (on_board yes)
-    (property "Reference" "C69" (id 0) (at 146.05 49.53 90)
+    (property "Reference" "C67" (id 0) (at 146.05 49.53 90)
       (effects (font (size 1 1)) (justify left))
     )
@@
   (symbol (lib_id "Device:R_Small") (at 81.28 125.73 90) (unit 1)
     (in_bom yes) (on_board yes)
-    (property "Reference" "R62" (id 0) (at 74.93 127 90)
+    (property "Reference" "R65" (id 0) (at 74.93 127 90)
       (effects (font (size 1 1)) (justify right))
     )
@@
   (symbol (lib_id "Device:R_Small") (at 99.06 100.33 90) (unit 1)
     (in_bom yes) (on_board yes)
-    (property "Reference" "R74" (id 0) (at 92.71 99.06 90)
+    (property "Reference" "R77" (id 0) (at 92.71 99.06 90)
       (effects (font (size 1 1)) (justify right))
     )
@@
   (symbol (lib_id "Device:C_Small") (at 147.32 160.02 90) (unit 1)
     (in_bom yes) (on_board yes)
-    (property "Reference" "C76" (id 0) (at 146.05 158.75 90)
+    (property "Reference" "C74" (id 0) (at 146.05 158.75 90)
       (effects (font (size 1 1)) (justify left))
     )
@@
   (symbol (lib_id "Device:R_Small") (at 99.06 85.09 90) (unit 1)
     (in_bom yes) (on_board yes)
-    (property "Reference" "R70" (id 0) (at 92.71 83.82 90)
+    (property "Reference" "R73" (id 0) (at 92.71 83.82 90)
       (effects (font (size 1 1)) (justify right))
     )
@@
   (symbol (lib_id "Device:R_Small") (at 99.06 92.71 90) (unit 1)
     (in_bom yes) (on_board yes)
-    (property "Reference" "R72" (id 0) (at 92.71 91.44 90)
-      (effects (font (size 1 1)) (justify right))
-    )
+    (property "Reference" "R75" (id 0) (at 92.71 91.44 90)
+      (effects (font (size 1 1)) (justify right))
+    )

Commit message: work on control logic
Parts:
- renumbered R64 to R66, R65 to R67, R66 to R68, R67 to R69, R68 to R70, R69 to R71, R70 to R72, R71 to R73, R72 to R74, R73 to R75, R74 to R76, R75 to R77, R76 to R78, R77 to R79
Changed lines of the file:
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@@
   (symbol (lib_id "Device:R_Small") (at 81.28 118.11 90) (unit 1)
     (in_bom yes) (on_board yes)
-    (property "Reference" "R64" (id 0) (at 74.93 116.84 90)
+    (property "Reference" "R66" (id 0) (at 74.93 116.84 90)
       (effects (font (size 1 1)) (justify right))
     )
@@
   (symbol (lib_id "Device:R_Small") (at 99.06 77.47 90) (unit 1)
     (in_bom yes) (on_board yes)
-    (property "Reference" "R71" (id 0) (at 92.71 76.2 90)
+    (property "Reference" "R73" (id 0) (at 92.71 76.2 90)
       (effects (font (size 1 1)) (justify right))
     )
@@
   (symbol (lib_id "Device:R_Small") (at 99.06 82.55 90) (unit 1)
     (in_bom yes) (on_board yes)
-    (property "Reference" "R72" (id 0) (at 92.71 81.28 90)
+    (property "Reference" "R74" (id 0) (at 92.71 81.28 90)
       (effects (font (size 1 1)) (justify right))
     )
@@
   (symbol (lib_id "Device:R_Small") (at 99.06 74.93 90) (unit 1)
     (in_bom yes) (on_board yes)
-    (property "Reference" "R70" (id 0) (at 92.71 73.66 90)
+    (property "Reference" "R72" (id 0) (at 92.71 73.66 90)
       (effects (font (size 1 1)) (justify right))
     )
@@
   (symbol (lib_id "Device:R_Small") (at 99.06 59.69 90) (unit 1)
     (in_bom yes) (on_board yes)
-    (property "Reference" "R66" (id 0) (at 93.345 58.801 90)
+    (property "Reference" "R68" (id 0) (at 93.345 58.801 90)
       (effects (font (size 1 1)) (justify right))
     )
@@
   (symbol (lib_id "Device:R_Small") (at 99.06 67.31 90) (unit 1)
     (in_bom yes) (on_board yes)
-    (property "Reference" "R68" (id 0) (at 92.71 66.04 90)
+    (property "Reference" "R70" (id 0) (at 92.71 66.04 90)
       (effects (font (size 1 1)) (justify right))
     )
@@
   (symbol (lib_id "Device:R_Small") (at 99.06 97.79 90) (unit 1)
     (in_bom yes) (on_board yes)
-    (property "Reference" "R76" (id 0) (at 92.71 96.52 90)
+    (property "Reference" "R78" (id 0) (at 92.71 96.52 90)
       (effects (font (size 1 1)) (justify right))
     )
@@
   (symbol (lib_id "Device:R_Small") (at 99.06 69.85 90) (unit 1)
     (in_bom yes) (on_board yes)
-    (property "Reference" "R69" (id 0) (at 92.71 68.58 90)
+    (property "Reference" "R71" (id 0) (at 92.71 68.58 90)
       (effects (font (size 1 1)) (justify right))
     )
@@
   (symbol (lib_id "Device:R_Small") (at 99.06 90.17 90) (unit 1)
     (in_bom yes) (on_board yes)
-    (property "Reference" "R74" (id 0) (at 92.71 88.9 90)
+    (property "Reference" "R76" (id 0) (at 92.71 88.9 90)
       (effects (font (size 1 1)) (justify right))
     )
@@
   (symbol (lib_id "Device:R_Small") (at 99.06 62.23 90) (unit 1)
     (in_bom yes) (on_board yes)
-    (property "Reference" "R67" (id 0) (at 92.71 60.96 90)
+    (property "Reference" "R69" (id 0) (at 92.71 60.96 90)
       (effects (font (size 1 1)) (justify right))
     )
@@
   (symbol (lib_id "Device:R_Small") (at 81.28 125.73 90) (unit 1)
     (in_bom yes) (on_board yes)
-    (property "Reference" "R65" (id 0) (at 74.93 127 90)
+    (property "Reference" "R67" (id 0) (at 74.93 127 90)
       (effects (font (size 1 1)) (justify right))
     )
@@
   (symbol (lib_id "Device:R_Small") (at 99.06 100.33 90) (unit 1)
     (in_bom yes) (on_board yes)
-    (property "Reference" "R77" (id 0) (at 92.71 99.06 90)
+    (property "Reference" "R79" (id 0) (at 92.71 99.06 90)
       (effects (font (size 1 1)) (justify right))
     )
@@
   (symbol (lib_id "Device:R_Small") (at 99.06 85.09 90) (unit 1)
     (in_bom yes) (on_board yes)
-    (property "Reference" "R73" (id 0) (at 92.71 83.82 90)
+    (property "Reference" "R75" (id 0) (at 92.71 83.82 90)
       (effects (font (size 1 1)) (justify right))
     )
@@
   (symbol (lib_id "Device:R_Small") (at 99.06 92.71 90) (unit 1)
     (in_bom yes) (on_board yes)
-    (property "Reference" "R75" (id 0) (at 92.71 91.44 90)
-      (effects (font (size 1 1)) (justify right))
-    )
+    (property "Reference" "R77" (id 0) (at 92.71 91.44 90)
+      (effects (font (size 1 1)) (justify right))
+    )

Commit message: work on control logic
Parts:
- renumbered C66 to C68, C67 to C69, C68 to C70, C69 to C71, C70 to C72, C71 to C73, C72 to C74, C73 to C75, C74 to C76, C75 to C77, C76 to C78, R66 to R69, R67 to R70, R68 to R71, R69 to R72, R70 to R73, R71 to R74, R72 to R75, R73 to R76, R74 to R77, R75 to R78, R76 to R79, R77 to R80, R78 to R81, R79 to R82
Changed lines of the file:
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@@
   (symbol (lib_id "Device:R_Small") (at 81.28 118.11 90) (unit 1)
     (in_bom yes) (on_board yes)
-    (property "Reference" "R66" (id 0) (at 74.93 116.84 90)
+    (property "Reference" "R69" (id 0) (at 74.93 116.84 90)
       (effects (font (size 1 1)) (justify right))
     )
@@
   (symbol (lib_id "Device:R_Small") (at 99.06 77.47 90) (unit 1)
     (in_bom yes) (on_board yes)
-    (property "Reference" "R73" (id 0) (at 92.71 76.2 90)
+    (property "Reference" "R76" (id 0) (at 92.71 76.2 90)
       (effects (font (size 1 1)) (justify right))
     )
@@
   (symbol (lib_id "Device:C_Small") (at 147.32 54.61 90) (unit 1)
     (in_bom yes) (on_board yes)
-    (property "Reference" "C68" (id 0) (at 146.05 53.34 90)
+    (property "Reference" "C70" (id 0) (at 146.05 53.34 90)
       (effects (font (size 1 1)) (justify left))
     )
@@
   (symbol (lib_id "Device:R_Small") (at 99.06 82.55 90) (unit 1)
     (in_bom yes) (on_board yes)
-    (property "Reference" "R74" (id 0) (at 92.71 81.28 90)
+    (property "Reference" "R77" (id 0) (at 92.71 81.28 90)
       (effects (font (size 1 1)) (justify right))
     )
@@
   (symbol (lib_id "Device:C_Small") (at 147.32 167.64 90) (unit 1)
     (in_bom yes) (on_board yes)
-    (property "Reference" "C76" (id 0) (at 146.05 166.37 90)
+    (property "Reference" "C78" (id 0) (at 146.05 166.37 90)
       (effects (font (size 1 1)) (justify left))
     )
@@
   (symbol (lib_id "Device:R_Small") (at 99.06 74.93 90) (unit 1)
     (in_bom yes) (on_board yes)
-    (property "Reference" "R72" (id 0) (at 92.71 73.66 90)
+    (property "Reference" "R75" (id 0) (at 92.71 73.66 90)
       (effects (font (size 1 1)) (justify right))
     )
@@
   (symbol (lib_id "Device:R_Small") (at 99.06 59.69 90) (unit 1)
     (in_bom yes) (on_board yes)
-    (property "Reference" "R68" (id 0) (at 93.345 58.801 90)
+    (property "Reference" "R71" (id 0) (at 93.345 58.801 90)
       (effects (font (size 1 1)) (justify right))
     )
@@
   (symbol (lib_id "Device:R_Small") (at 99.06 67.31 90) (unit 1)
     (in_bom yes) (on_board yes)
-    (property "Reference" "R70" (id 0) (at 92.71 66.04 90)
+    (property "Reference" "R73" (id 0) (at 92.71 66.04 90)
       (effects (font (size 1 1)) (justify right))
     )
@@
   (symbol (lib_id "Device:C_Small") (at 147.32 152.4 90) (unit 1)
     (in_bom yes) (on_board yes)
-    (property "Reference" "C72" (id 0) (at 146.05 151.13 90)
+    (property "Reference" "C74" (id 0) (at 146.05 151.13 90)
       (effects (font (size 1 1)) (justify left))
     )
@@
   (symbol (lib_id "Device:C_Small") (at 147.32 144.78 90) (unit 1)
     (in_bom yes) (on_board yes)
-    (property "Reference" "C70" (id 0) (at 146.05 143.51 90)
+    (property "Reference" "C72" (id 0) (at 146.05 143.51 90)
       (effects (font (size 1 1)) (justify left))
     )
@@
   (symbol (lib_id "Device:C_Small") (at 147.32 140.97 90) (unit 1)
     (in_bom yes) (on_board yes)
-    (property "Reference" "C69" (id 0) (at 146.05 139.7 90)
+    (property "Reference" "C71" (id 0) (at 146.05 139.7 90)
       (effects (font (size 1 1)) (justify left))
     )
@@
   (symbol (lib_id "Device:R_Small") (at 99.06 97.79 90) (unit 1)
     (in_bom yes) (on_board yes)
-    (property "Reference" "R78" (id 0) (at 92.71 96.52 90)
+    (property "Reference" "R81" (id 0) (at 92.71 96.52 90)
       (effects (font (size 1 1)) (justify right))
     )
@@
   (symbol (lib_id "Device:C_Small") (at 147.32 148.59 90) (unit 1)
     (in_bom yes) (on_board yes)
-    (property "Reference" "C71" (id 0) (at 146.05 147.32 90)
+    (property "Reference" "C73" (id 0) (at 146.05 147.32 90)
       (effects (font (size 1 1)) (justify left))
     )
@@
   (symbol (lib_id "Device:C_Small") (at 147.32 46.99 90) (unit 1)
     (in_bom yes) (on_board yes)
-    (property "Reference" "C66" (id 0) (at 146.05 45.72 90)
+    (property "Reference" "C68" (id 0) (at 146.05 45.72 90)
       (effects (font (size 1 1)) (justify left))
     )
@@
   (symbol (lib_id "power:GND") (at 90.17 153.67 0) (unit 1)
     (in_bom yes) (on_board yes)
-    (property "Reference" "#PWR055" (id 0) (at 90.17 160.02 0)
+    (property "Reference" "#PWR056" (id 0) (at 90.17 160.02 0)
       (effects (font (size 1.27 1.27)) hide)
     )
@@
   (symbol (lib_id "power:GND") (at 154.94 170.18 0) (unit 1)
     (in_bom yes) (on_board yes)
-    (property "Reference" "#PWR057" (id 0) (at 154.94 176.53 0)
+    (property "Reference" "#PWR058" (id 0) (at 154.94 176.53 0)
       (effects (font (size 1.27 1.27)) hide)
     )
@@
   (symbol (lib_id "Device:R_Small") (at 99.06 69.85 90) (unit 1)
     (in_bom yes) (on_board yes)
-    (property "Reference" "R71" (id 0) (at 92.71 68.58 90)
+    (property "Reference" "R74" (id 0) (at 92.71 68.58 90)
       (effects (font (size 1 1)) (justify right))
     )
@@
   (symbol (lib_id "Device:C_Small") (at 147.32 163.83 90) (unit 1)
     (in_bom yes) (on_board yes)
-    (property "Reference" "C75" (id 0) (at 146.05 162.56 90)
+    (property "Reference" "C77" (id 0) (at 146.05 162.56 90)
       (effects (font (size 1 1)) (justify left))
     )
@@
   (symbol (lib_id "Device:C_Small") (at 147.32 156.21 90) (unit 1)
     (in_bom yes) (on_board yes)
-    (property "Reference" "C73" (id 0) (at 146.05 154.94 90)
+    (property "Reference" "C75" (id 0) (at 146.05 154.94 90)
       (effects (font (size 1 1)) (justify left))
     )
@@
   (symbol (lib_id "power:GND") (at 154.94 57.15 0) (unit 1)
     (in_bom yes) (on_board yes)
-    (property "Reference" "#PWR056" (id 0) (at 154.94 63.5 0)
+    (property "Reference" "#PWR057" (id 0) (at 154.94 63.5 0)
       (effects (font (size 1.27 1.27)) hide)
     )
@@
   (symbol (lib_id "Device:R_Small") (at 99.06 90.17 90) (unit 1)
     (in_bom yes) (on_board yes)
-    (property "Reference" "R76" (id 0) (at 92.71 88.9 90)
+    (property "Reference" "R79" (id 0) (at 92.71 88.9 90)
       (effects (font (size 1 1)) (justify right))
     )
@@
   (symbol (lib_id "Device:R_Small") (at 99.06 62.23 90) (unit 1)
     (in_bom yes) (on_board yes)
-    (property "Reference" "R69" (id 0) (at 92.71 60.96 90)
+    (property "Reference" "R72" (id 0) (at 92.71 60.96 90)
       (effects (font (size 1 1)) (justify right))
     )
@@
   (symbol (lib_id "Device:C_Small") (at 147.32 50.8 90) (unit 1)
     (in_bom yes) (on_board yes)
-    (property "Reference" "C67" (id 0) (at 146.05 49.53 90)
+    (property "Reference" "C69" (id 0) (at 146.05 49.53 90)
       (effects (font (size 1 1)) (justify left))
     )
@@
   (symbol (lib_id "Device:R_Small") (at 81.28 125.73 90) (unit 1)
     (in_bom yes) (on_board yes)
-    (property "Reference" "R67" (id 0) (at 74.93 127 90)
+    (property "Reference" "R70" (id 0) (at 74.93 127 90)
       (effects (font (size 1 1)) (justify right))
     )
@@
   (symbol (lib_id "Device:R_Small") (at 99.06 100.33 90) (unit 1)
     (in_bom yes) (on_board yes)
-    (property "Reference" "R79" (id 0) (at 92.71 99.06 90)
+    (property "Reference" "R82" (id 0) (at 92.71 99.06 90)
       (effects (font (size 1 1)) (justify right))
     )
@@
   (symbol (lib_id "Device:C_Small") (at 147.32 160.02 90) (unit 1)
     (in_bom yes) (on_board yes)
-    (property "Reference" "C74" (id 0) (at 146.05 158.75 90)
+    (property "Reference" "C76" (id 0) (at 146.05 158.75 90)
       (effects (font (size 1 1)) (justify left))
     )
@@
   (symbol (lib_id "Device:R_Small") (at 99.06 85.09 90) (unit 1)
     (in_bom yes) (on_board yes)
-    (property "Reference" "R75" (id 0) (at 92.71 83.82 90)
+    (property "Reference" "R78" (id 0) (at 92.71 83.82 90)
       (effects (font (size 1 1)) (justify right))
     )
@@
   (symbol (lib_id "Device:R_Small") (at 99.06 92.71 90) (unit 1)
     (in_bom yes) (on_board yes)
-    (property "Reference" "R77" (id 0) (at 92.71 91.44 90)
-      (effects (font (size 1 1)) (justify right))
-    )
+    (property "Reference" "R80" (id 0) (at 92.71 91.44 90)
+      (effects (font (size 1 1)) (justify right))
+    )

Commit message: layout experiments
Connections:
- net GND: now also J8.S (SHIELD); no longer J8.S1 (SHIELD), J8.S2 (SHIELD)
Changed lines of the file:
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@@
   (junction (at 90.17 69.85) (diameter 0.9144) (color 0 0 0 0)
-  )
-  (junction (at 90.17 148.59) (diameter 0.9144) (color 0 0 0 0)
   )
   (junction (at 154.94 156.21) (diameter 0.9144) (color 0 0 0 0)
@@
     (stroke (width 0) (type solid) (color 0 0 0 0))
   )
-  (wire (pts (xy 90.17 143.51) (xy 90.17 148.59))
+  (wire (pts (xy 90.17 143.51) (xy 90.17 153.67))
     (stroke (width 0) (type solid) (color 0 0 0 0))
   )
@@
   )
   (wire (pts (xy 101.6 59.69) (xy 105.41 59.69))
-    (stroke (width 0) (type solid) (color 0 0 0 0))
-  )
-  (wire (pts (xy 90.17 148.59) (xy 90.17 153.67))
     (stroke (width 0) (type solid) (color 0 0 0 0))
   )
@@
   )
   (wire (pts (xy 90.17 69.85) (xy 96.52 69.85))
-    (stroke (width 0) (type solid) (color 0 0 0 0))
-  )
-  (wire (pts (xy 90.17 148.59) (xy 105.41 148.59))
     (stroke (width 0) (type solid) (color 0 0 0 0))
   )
@@
       (effects (font (size 1.27 1.27)) (justify left bottom))
     )
-    (property "Value" "1-2199119-6" (id 1) (at 111.76 153.67 0)
+    (property "Value" "1-2199119-6" (id 1) (at 111.125 153.67 0)
       (effects (font (size 1.27 1.27)) (justify left bottom))
     )
@@
     (pin "8")
     (pin "9")
-    (pin "S1")
-    (pin "S2")
+    (pin "S")
   )
   (symbol (lib_id "power:GND") (at 154.94 57.15 0) (unit 1)
