File: psugroup.kicad_sch (KiCad schematic)
At the start: 0 parts

Commit message: leds
Other:
- sheet +3.3V PSU ports: added +3.3V_OK; removed none
- sheet +5V PSU ports: added +5V_OK; removed none
Changed lines of the file:
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@@
     (stroke (width 0) (type solid) (color 0 0 0 0))
+  )
+  (wire (pts (xy 139.7 134.62) (xy 144.78 134.62))
+    (stroke (width 0) (type default) (color 0 0 0 0))
   )
   (wire (pts (xy 170.18 129.54) (xy 179.07 129.54))
@@
   )
   (wire (pts (xy 219.71 78.74) (xy 213.36 78.74))
+    (stroke (width 0) (type default) (color 0 0 0 0))
+  )
+  (wire (pts (xy 139.7 91.44) (xy 144.78 91.44))
     (stroke (width 0) (type default) (color 0 0 0 0))
   )
@@
     (effects (font (size 1.27 1.27)) (justify right))
   )
+  (hierarchical_label "+3.3V_OK" (shape output) (at 144.78 91.44 0)
+    (effects (font (size 1.27 1.27)) (justify left))
+  )
   (hierarchical_label "+12V_IN" (shape input) (at 82.55 78.74 180)
     (effects (font (size 1.27 1.27)) (justify right))
   )
   (hierarchical_label "ALERT_+3.3V" (shape output) (at 219.71 81.28 0)
+    (effects (font (size 1.27 1.27)) (justify left))
+  )
+  (hierarchical_label "+5V_OK" (shape output) (at 144.78 134.62 0)
     (effects (font (size 1.27 1.27)) (justify left))
   )
@@
       (effects (font (size 1.27 1.27)) (justify right))
     )
+    (pin "+5V_OK" output (at 139.7 134.62 0)
+      (effects (font (size 1.27 1.27)) (justify right))
+    )
   )
   (sheet (at 107.95 76.2) (size 31.75 17.78) (fields_autoplaced)
@@
       (effects (font (size 1.27 1.27)) (justify left))
     )
+    (pin "+3.3V_OK" output (at 139.7 91.44 0)
+      (effects (font (size 1.27 1.27)) (justify right))
+    )
   )
