File: cm4usb.kicad_sch (KiCad schematic)
At the start: 24 parts, among them J6 USB4110-GF-A, J7 USB4110-GF-A, U14 USB3740B-AI2, U15 AP22653FDZ-7

Commit message: board refresh
Parts:
- renumbered C26 to C24, C27 to C25, C28 to C26, C29 to C27, C30 to C28, C31 to C29, C32 to C30, C33 to C31, C34 to C32, C35 to C33, R42 to R45, R43 to R46, R44 to R47, R45 to R48, R46 to R49, R47 to R50, R48 to R51, R49 to R52, R50 to R53, U14 to U13, U15 to U14
Changed lines of the file:
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@@
   (symbol (lib_id "Device:R_Small") (at 297.434 85.344 270) (unit 1)
     (in_bom yes) (on_board yes)
-    (property "Reference" "R49" (id 0) (at 297.434 87.63 90))
+    (property "Reference" "R52" (id 0) (at 297.434 87.63 90))
     (property "Value" "10k" (id 1) (at 297.434 90.17 90))
     (property "Footprint" "Resistor_SMD:R_0402_1005Metric" (id 2) (at 297.434 85.344 0)
@@
   (symbol (lib_id "Device:R_Small") (at 203.2 254 90) (unit 1)
     (in_bom yes) (on_board yes)
-    (property "Reference" "R47" (id 0) (at 196.85 252.73 90)
+    (property "Reference" "R50" (id 0) (at 196.85 252.73 90)
       (effects (font (size 1.27 1.27)) (justify right))
     )
@@
   (symbol (lib_id "Device:C_Small") (at 337.82 82.55 0) (unit 1)
     (in_bom yes) (on_board yes)
-    (property "Reference" "C32" (id 0) (at 339.09 81.28 0)
+    (property "Reference" "C30" (id 0) (at 339.09 81.28 0)
       (effects (font (size 1.27 1.27)) (justify left))
     )
@@
   (symbol (lib_id "Device:R_Small") (at 142.24 128.27 90) (unit 1)
     (in_bom yes) (on_board yes)
-    (property "Reference" "R45" (id 0) (at 145.034 131.064 90)
+    (property "Reference" "R48" (id 0) (at 145.034 131.064 90)
       (effects (font (size 1.27 1.27)) (justify left))
     )
@@
   (symbol (lib_id "Device:C_Small") (at 327.66 82.55 0) (unit 1)
     (in_bom yes) (on_board yes)
-    (property "Reference" "C31" (id 0) (at 328.93 81.28 0)
+    (property "Reference" "C29" (id 0) (at 328.93 81.28 0)
       (effects (font (size 1.27 1.27)) (justify left))
     )
@@
   (symbol (lib_id "power:GND") (at 368.3 94.742 0) (unit 1)
     (in_bom yes) (on_board yes)
-    (property "Reference" "#PWR044" (id 0) (at 368.3 101.092 0)
+    (property "Reference" "#PWR042" (id 0) (at 368.3 101.092 0)
       (effects (font (size 1.27 1.27)) hide)
     )
@@
   (symbol (lib_id "Device:R_Small") (at 142.24 87.63 270) (unit 1)
     (in_bom yes) (on_board yes)
-    (property "Reference" "R44" (id 0) (at 139.7 82.55 90)
+    (property "Reference" "R47" (id 0) (at 139.7 82.55 90)
       (effects (font (size 1.27 1.27)) (justify left))
     )
@@
   (symbol (lib_id "Device:C_Small") (at 347.98 82.55 0) (unit 1)
     (in_bom yes) (on_board yes)
-    (property "Reference" "C33" (id 0) (at 349.25 81.28 0)
+    (property "Reference" "C31" (id 0) (at 349.25 81.28 0)
       (effects (font (size 1.27 1.27)) (justify left))
     )
@@
   (symbol (lib_id "Device:C_Small") (at 358.14 82.55 0) (unit 1)
     (in_bom yes) (on_board yes)
-    (property "Reference" "C34" (id 0) (at 359.41 81.28 0)
+    (property "Reference" "C32" (id 0) (at 359.41 81.28 0)
       (effects (font (size 1.27 1.27)) (justify left))
     )
@@
   (symbol (lib_id "Device:C_Small") (at 203.2 259.08 90) (unit 1)
     (in_bom yes) (on_board yes)
-    (property "Reference" "C29" (id 0) (at 196.85 257.81 90)
+    (property "Reference" "C27" (id 0) (at 196.85 257.81 90)
       (effects (font (size 1.27 1.27)) (justify right))
     )
@@
   (symbol (lib_id "Device:C_Small") (at 368.3 82.55 0) (unit 1)
     (in_bom yes) (on_board yes)
-    (property "Reference" "C35" (id 0) (at 369.57 81.28 0)
+    (property "Reference" "C33" (id 0) (at 369.57 81.28 0)
       (effects (font (size 1.27 1.27)) (justify left))
     )
@@
   (symbol (lib_id "power:GND") (at 106.68 151.13 0) (unit 1)
     (in_bom yes) (on_board yes)
-    (property "Reference" "#PWR041" (id 0) (at 106.68 157.48 0)
+    (property "Reference" "#PWR039" (id 0) (at 106.68 157.48 0)
       (effects (font (size 1.27 1.27)) hide)
     )
@@
   (symbol (lib_id "Device:R_Small") (at 207.01 218.44 90) (unit 1)
     (in_bom yes) (on_board yes)
-    (property "Reference" "R48" (id 0) (at 201.93 217.17 90))
+    (property "Reference" "R51" (id 0) (at 201.93 217.17 90))
     (property "Value" "5.1k" (id 1) (at 212.09 217.17 90))
     (property "Footprint" "Resistor_SMD:R_0402_1005Metric" (id 2) (at 207.01 218.44 0)
@@
   (symbol (lib_id "Device:R_Small") (at 80.01 254 90) (unit 1)
     (in_bom yes) (on_board yes)
-    (property "Reference" "R42" (id 0) (at 73.66 252.73 90)
+    (property "Reference" "R45" (id 0) (at 73.66 252.73 90)
       (effects (font (size 1.27 1.27)) (justify right))
     )
@@
   (symbol (lib_id "Device:R_Small") (at 82.55 218.44 90) (unit 1)
     (in_bom yes) (on_board yes)
-    (property "Reference" "R43" (id 0) (at 77.47 217.17 90))
+    (property "Reference" "R46" (id 0) (at 77.47 217.17 90))
     (property "Value" "5.1k" (id 1) (at 87.63 217.17 90))
     (property "Footprint" "Resistor_SMD:R_0402_1005Metric" (id 2) (at 82.55 218.44 0)
@@
   (symbol (lib_id "power:GND") (at 95.25 262.89 0) (unit 1)
     (in_bom yes) (on_board yes)
-    (property "Reference" "#PWR040" (id 0) (at 95.25 269.24 0)
+    (property "Reference" "#PWR038" (id 0) (at 95.25 269.24 0)
       (effects (font (size 1.27 1.27)) hide)
     )
@@
   (symbol (lib_id "power:GND") (at 149.86 151.13 0) (unit 1)
     (in_bom yes) (on_board yes)
-    (property "Reference" "#PWR042" (id 0) (at 149.86 157.48 0)
+    (property "Reference" "#PWR040" (id 0) (at 149.86 157.48 0)
       (effects (font (size 1.27 1.27)) hide)
     )
@@
   (symbol (lib_id "Power_Protection_Diodes:AP22653FDZ-7") (at 297.18 78.74 0) (unit 1)
     (in_bom yes) (on_board yes)
-    (property "Reference" "U15" (id 0) (at 297.18 69.85 0))
+    (property "Reference" "U14" (id 0) (at 297.18 69.85 0))
     (property "Value" "AP22653FDZ-7" (id 1) (at 297.18 72.39 0))
     (property "Footprint" "Power_Protection_Diodes:Diodes_W-DFN2020-6_A1" (id 2) (at 297.18 92.71 0)
@@
   (symbol (lib_id "Interface_USB_Microchip:USB3740B-AI2") (at 121.285 116.84 0) (unit 1)
     (in_bom yes) (on_board yes)
-    (property "Reference" "U14" (id 0) (at 121.92 102.87 0))
+    (property "Reference" "U13" (id 0) (at 121.92 102.87 0))
     (property "Value" "USB3740B-AI2" (id 1) (at 121.92 105.41 0))
     (property "Footprint" "Interface_USB_Microchip:Microchip_UQFN-10_1.3x1.8mm_P0.4mm_pin1" (id 2) (at 121.285 149.86 0)
@@
   (symbol (lib_id "Device:C_Small") (at 80.01 259.08 90) (unit 1)
     (in_bom yes) (on_board yes)
-    (property "Reference" "C26" (id 0) (at 73.66 257.81 90)
+    (property "Reference" "C24" (id 0) (at 73.66 257.81 90)
       (effects (font (size 1.27 1.27)) (justify right))
     )
@@
   (symbol (lib_id "Device:C_Small") (at 85.09 130.81 0) (mirror y) (unit 1)
     (in_bom yes) (on_board yes) (fields_autoplaced)
-    (property "Reference" "C27" (id 0) (at 82.55 129.54 0)
+    (property "Reference" "C25" (id 0) (at 82.55 129.54 0)
       (effects (font (size 1.27 1.27)) (justify left))
     )
@@
   (symbol (lib_id "Device:R_Small") (at 316.23 78.74 90) (unit 1)
     (in_bom yes) (on_board yes)
-    (property "Reference" "R50" (id 0) (at 318.77 81.28 90)
+    (property "Reference" "R53" (id 0) (at 318.77 81.28 90)
       (effects (font (size 1.27 1.27)) (justify left))
     )
@@
   (symbol (lib_id "power:GND") (at 219.71 262.89 0) (unit 1)
     (in_bom yes) (on_board yes)
-    (property "Reference" "#PWR043" (id 0) (at 219.71 269.24 0)
+    (property "Reference" "#PWR041" (id 0) (at 219.71 269.24 0)
       (effects (font (size 1.27 1.27)) hide)
     )
@@
   (symbol (lib_id "Device:C_Small") (at 267.97 81.28 0) (unit 1)
     (in_bom yes) (on_board yes)
-    (property "Reference" "C30" (id 0) (at 269.24 80.01 0)
+    (property "Reference" "C28" (id 0) (at 269.24 80.01 0)
       (effects (font (size 1.27 1.27)) (justify left))
     )
@@
   (symbol (lib_id "Device:C_Small") (at 96.52 130.81 0) (mirror y) (unit 1)
     (in_bom yes) (on_board yes) (fields_autoplaced)
-    (property "Reference" "C28" (id 0) (at 93.98 129.54 0)
+    (property "Reference" "C26" (id 0) (at 93.98 129.54 0)
       (effects (font (size 1.27 1.27)) (justify left))
     )
@@
   (symbol (lib_id "Device:R_Small") (at 149.86 92.71 0) (mirror x) (unit 1)
     (in_bom yes) (on_board yes)
-    (property "Reference" "R46" (id 0) (at 151.384 91.44 0)
+    (property "Reference" "R49" (id 0) (at 151.384 91.44 0)
       (effects (font (size 1.27 1.27)) (justify left))
     )
@@
   (symbol (lib_id "power:GND") (at 85.09 138.43 0) (mirror y) (unit 1)
     (in_bom yes) (on_board yes)
-    (property "Reference" "#PWR039" (id 0) (at 85.09 144.78 0)
-      (effects (font (size 1.27 1.27)) hide)
-    )
+    (property "Reference" "#PWR037" (id 0) (at 85.09 144.78 0)
+      (effects (font (size 1.27 1.27)) hide)
+    )

Commit message: work on control logic
Parts:
- renumbered R45 to R47, R46 to R48, R47 to R49, R48 to R50, R49 to R51, R50 to R52, R51 to R53, R52 to R54, R53 to R55
Changed lines of the file:
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@@
   (symbol (lib_id "Device:R_Small") (at 297.434 85.344 270) (unit 1)
     (in_bom yes) (on_board yes)
-    (property "Reference" "R52" (id 0) (at 297.434 87.63 90))
+    (property "Reference" "R54" (id 0) (at 297.434 87.63 90))
     (property "Value" "10k" (id 1) (at 297.434 90.17 90))
     (property "Footprint" "Resistor_SMD:R_0402_1005Metric" (id 2) (at 297.434 85.344 0)
@@
   (symbol (lib_id "Device:R_Small") (at 203.2 254 90) (unit 1)
     (in_bom yes) (on_board yes)
-    (property "Reference" "R50" (id 0) (at 196.85 252.73 90)
+    (property "Reference" "R52" (id 0) (at 196.85 252.73 90)
       (effects (font (size 1.27 1.27)) (justify right))
     )
@@
   (symbol (lib_id "Device:R_Small") (at 142.24 128.27 90) (unit 1)
     (in_bom yes) (on_board yes)
-    (property "Reference" "R48" (id 0) (at 145.034 131.064 90)
+    (property "Reference" "R50" (id 0) (at 145.034 131.064 90)
       (effects (font (size 1.27 1.27)) (justify left))
     )
@@
   (symbol (lib_id "Device:R_Small") (at 142.24 87.63 270) (unit 1)
     (in_bom yes) (on_board yes)
-    (property "Reference" "R47" (id 0) (at 139.7 82.55 90)
+    (property "Reference" "R49" (id 0) (at 139.7 82.55 90)
       (effects (font (size 1.27 1.27)) (justify left))
     )
@@
   (symbol (lib_id "Device:R_Small") (at 207.01 218.44 90) (unit 1)
     (in_bom yes) (on_board yes)
-    (property "Reference" "R51" (id 0) (at 201.93 217.17 90))
+    (property "Reference" "R53" (id 0) (at 201.93 217.17 90))
     (property "Value" "5.1k" (id 1) (at 212.09 217.17 90))
     (property "Footprint" "Resistor_SMD:R_0402_1005Metric" (id 2) (at 207.01 218.44 0)
@@
   (symbol (lib_id "Device:R_Small") (at 80.01 254 90) (unit 1)
     (in_bom yes) (on_board yes)
-    (property "Reference" "R45" (id 0) (at 73.66 252.73 90)
+    (property "Reference" "R47" (id 0) (at 73.66 252.73 90)
       (effects (font (size 1.27 1.27)) (justify right))
     )
@@
   (symbol (lib_id "Device:R_Small") (at 82.55 218.44 90) (unit 1)
     (in_bom yes) (on_board yes)
-    (property "Reference" "R46" (id 0) (at 77.47 217.17 90))
+    (property "Reference" "R48" (id 0) (at 77.47 217.17 90))
     (property "Value" "5.1k" (id 1) (at 87.63 217.17 90))
     (property "Footprint" "Resistor_SMD:R_0402_1005Metric" (id 2) (at 82.55 218.44 0)
@@
   (symbol (lib_id "Device:R_Small") (at 316.23 78.74 90) (unit 1)
     (in_bom yes) (on_board yes)
-    (property "Reference" "R53" (id 0) (at 318.77 81.28 90)
+    (property "Reference" "R55" (id 0) (at 318.77 81.28 90)
       (effects (font (size 1.27 1.27)) (justify left))
     )
@@
   (symbol (lib_id "Device:R_Small") (at 149.86 92.71 0) (mirror x) (unit 1)
     (in_bom yes) (on_board yes)
-    (property "Reference" "R49" (id 0) (at 151.384 91.44 0)
-      (effects (font (size 1.27 1.27)) (justify left))
-    )
+    (property "Reference" "R51" (id 0) (at 151.384 91.44 0)
+      (effects (font (size 1.27 1.27)) (justify left))
+    )

Commit message: work on control logic
Parts:
- renumbered C24 to C26, C25 to C27, C26 to C28, C27 to C29, C28 to C30, C29 to C31, C30 to C32, C31 to C33, C32 to C34, C33 to C35, R47 to R50, R48 to R51, R49 to R52, R50 to R53, R51 to R54, R52 to R55, R53 to R56, R54 to R57, R55 to R58, U13 to U14, U14 to U15
Changed lines of the file:
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@@
   (symbol (lib_id "Device:R_Small") (at 297.434 85.344 270) (unit 1)
     (in_bom yes) (on_board yes)
-    (property "Reference" "R54" (id 0) (at 297.434 87.63 90))
+    (property "Reference" "R57" (id 0) (at 297.434 87.63 90))
     (property "Value" "10k" (id 1) (at 297.434 90.17 90))
     (property "Footprint" "Resistor_SMD:R_0402_1005Metric" (id 2) (at 297.434 85.344 0)
@@
   (symbol (lib_id "Device:R_Small") (at 203.2 254 90) (unit 1)
     (in_bom yes) (on_board yes)
-    (property "Reference" "R52" (id 0) (at 196.85 252.73 90)
+    (property "Reference" "R55" (id 0) (at 196.85 252.73 90)
       (effects (font (size 1.27 1.27)) (justify right))
     )
@@
   (symbol (lib_id "Device:C_Small") (at 337.82 82.55 0) (unit 1)
     (in_bom yes) (on_board yes)
-    (property "Reference" "C30" (id 0) (at 339.09 81.28 0)
+    (property "Reference" "C32" (id 0) (at 339.09 81.28 0)
       (effects (font (size 1.27 1.27)) (justify left))
     )
@@
   (symbol (lib_id "Device:R_Small") (at 142.24 128.27 90) (unit 1)
     (in_bom yes) (on_board yes)
-    (property "Reference" "R50" (id 0) (at 145.034 131.064 90)
+    (property "Reference" "R53" (id 0) (at 145.034 131.064 90)
       (effects (font (size 1.27 1.27)) (justify left))
     )
@@
   (symbol (lib_id "Device:C_Small") (at 327.66 82.55 0) (unit 1)
     (in_bom yes) (on_board yes)
-    (property "Reference" "C29" (id 0) (at 328.93 81.28 0)
+    (property "Reference" "C31" (id 0) (at 328.93 81.28 0)
       (effects (font (size 1.27 1.27)) (justify left))
     )
@@
   (symbol (lib_id "power:GND") (at 368.3 94.742 0) (unit 1)
     (in_bom yes) (on_board yes)
-    (property "Reference" "#PWR042" (id 0) (at 368.3 101.092 0)
+    (property "Reference" "#PWR043" (id 0) (at 368.3 101.092 0)
       (effects (font (size 1.27 1.27)) hide)
     )
@@
   (symbol (lib_id "Device:R_Small") (at 142.24 87.63 270) (unit 1)
     (in_bom yes) (on_board yes)
-    (property "Reference" "R49" (id 0) (at 139.7 82.55 90)
+    (property "Reference" "R52" (id 0) (at 139.7 82.55 90)
       (effects (font (size 1.27 1.27)) (justify left))
     )
@@
   (symbol (lib_id "Device:C_Small") (at 347.98 82.55 0) (unit 1)
     (in_bom yes) (on_board yes)
-    (property "Reference" "C31" (id 0) (at 349.25 81.28 0)
+    (property "Reference" "C33" (id 0) (at 349.25 81.28 0)
       (effects (font (size 1.27 1.27)) (justify left))
     )
@@
   (symbol (lib_id "Device:C_Small") (at 358.14 82.55 0) (unit 1)
     (in_bom yes) (on_board yes)
-    (property "Reference" "C32" (id 0) (at 359.41 81.28 0)
+    (property "Reference" "C34" (id 0) (at 359.41 81.28 0)
       (effects (font (size 1.27 1.27)) (justify left))
     )
@@
   (symbol (lib_id "Device:C_Small") (at 203.2 259.08 90) (unit 1)
     (in_bom yes) (on_board yes)
-    (property "Reference" "C27" (id 0) (at 196.85 257.81 90)
+    (property "Reference" "C29" (id 0) (at 196.85 257.81 90)
       (effects (font (size 1.27 1.27)) (justify right))
     )
@@
   (symbol (lib_id "Device:C_Small") (at 368.3 82.55 0) (unit 1)
     (in_bom yes) (on_board yes)
-    (property "Reference" "C33" (id 0) (at 369.57 81.28 0)
+    (property "Reference" "C35" (id 0) (at 369.57 81.28 0)
       (effects (font (size 1.27 1.27)) (justify left))
     )
@@
   (symbol (lib_id "power:GND") (at 106.68 151.13 0) (unit 1)
     (in_bom yes) (on_board yes)
-    (property "Reference" "#PWR039" (id 0) (at 106.68 157.48 0)
+    (property "Reference" "#PWR040" (id 0) (at 106.68 157.48 0)
       (effects (font (size 1.27 1.27)) hide)
     )
@@
   (symbol (lib_id "Device:R_Small") (at 207.01 218.44 90) (unit 1)
     (in_bom yes) (on_board yes)
-    (property "Reference" "R53" (id 0) (at 201.93 217.17 90))
+    (property "Reference" "R56" (id 0) (at 201.93 217.17 90))
     (property "Value" "5.1k" (id 1) (at 212.09 217.17 90))
     (property "Footprint" "Resistor_SMD:R_0402_1005Metric" (id 2) (at 207.01 218.44 0)
@@
   (symbol (lib_id "Device:R_Small") (at 80.01 254 90) (unit 1)
     (in_bom yes) (on_board yes)
-    (property "Reference" "R47" (id 0) (at 73.66 252.73 90)
+    (property "Reference" "R50" (id 0) (at 73.66 252.73 90)
       (effects (font (size 1.27 1.27)) (justify right))
     )
@@
   (symbol (lib_id "Device:R_Small") (at 82.55 218.44 90) (unit 1)
     (in_bom yes) (on_board yes)
-    (property "Reference" "R48" (id 0) (at 77.47 217.17 90))
+    (property "Reference" "R51" (id 0) (at 77.47 217.17 90))
     (property "Value" "5.1k" (id 1) (at 87.63 217.17 90))
     (property "Footprint" "Resistor_SMD:R_0402_1005Metric" (id 2) (at 82.55 218.44 0)
@@
   (symbol (lib_id "power:GND") (at 95.25 262.89 0) (unit 1)
     (in_bom yes) (on_board yes)
-    (property "Reference" "#PWR038" (id 0) (at 95.25 269.24 0)
+    (property "Reference" "#PWR039" (id 0) (at 95.25 269.24 0)
       (effects (font (size 1.27 1.27)) hide)
     )
@@
   (symbol (lib_id "power:GND") (at 149.86 151.13 0) (unit 1)
     (in_bom yes) (on_board yes)
-    (property "Reference" "#PWR040" (id 0) (at 149.86 157.48 0)
+    (property "Reference" "#PWR041" (id 0) (at 149.86 157.48 0)
       (effects (font (size 1.27 1.27)) hide)
     )
@@
   (symbol (lib_id "Power_Protection_Diodes:AP22653FDZ-7") (at 297.18 78.74 0) (unit 1)
     (in_bom yes) (on_board yes)
-    (property "Reference" "U14" (id 0) (at 297.18 69.85 0))
+    (property "Reference" "U15" (id 0) (at 297.18 69.85 0))
     (property "Value" "AP22653FDZ-7" (id 1) (at 297.18 72.39 0))
     (property "Footprint" "Power_Protection_Diodes:Diodes_W-DFN2020-6_A1" (id 2) (at 297.18 92.71 0)
@@
   (symbol (lib_id "Interface_USB_Microchip:USB3740B-AI2") (at 121.285 116.84 0) (unit 1)
     (in_bom yes) (on_board yes)
-    (property "Reference" "U13" (id 0) (at 121.92 102.87 0))
+    (property "Reference" "U14" (id 0) (at 121.92 102.87 0))
     (property "Value" "USB3740B-AI2" (id 1) (at 121.92 105.41 0))
     (property "Footprint" "Interface_USB_Microchip:Microchip_UQFN-10_1.3x1.8mm_P0.4mm_pin1" (id 2) (at 121.285 149.86 0)
@@
   (symbol (lib_id "Device:C_Small") (at 80.01 259.08 90) (unit 1)
     (in_bom yes) (on_board yes)
-    (property "Reference" "C24" (id 0) (at 73.66 257.81 90)
+    (property "Reference" "C26" (id 0) (at 73.66 257.81 90)
       (effects (font (size 1.27 1.27)) (justify right))
     )
@@
   (symbol (lib_id "Device:C_Small") (at 85.09 130.81 0) (mirror y) (unit 1)
     (in_bom yes) (on_board yes) (fields_autoplaced)
-    (property "Reference" "C25" (id 0) (at 82.55 129.54 0)
+    (property "Reference" "C27" (id 0) (at 82.55 129.54 0)
       (effects (font (size 1.27 1.27)) (justify left))
     )
@@
   (symbol (lib_id "Device:R_Small") (at 316.23 78.74 90) (unit 1)
     (in_bom yes) (on_board yes)
-    (property "Reference" "R55" (id 0) (at 318.77 81.28 90)
+    (property "Reference" "R58" (id 0) (at 318.77 81.28 90)
       (effects (font (size 1.27 1.27)) (justify left))
     )
@@
   (symbol (lib_id "power:GND") (at 219.71 262.89 0) (unit 1)
     (in_bom yes) (on_board yes)
-    (property "Reference" "#PWR041" (id 0) (at 219.71 269.24 0)
+    (property "Reference" "#PWR042" (id 0) (at 219.71 269.24 0)
       (effects (font (size 1.27 1.27)) hide)
     )
@@
   (symbol (lib_id "Device:C_Small") (at 267.97 81.28 0) (unit 1)
     (in_bom yes) (on_board yes)
-    (property "Reference" "C28" (id 0) (at 269.24 80.01 0)
+    (property "Reference" "C30" (id 0) (at 269.24 80.01 0)
       (effects (font (size 1.27 1.27)) (justify left))
     )
@@
   (symbol (lib_id "Device:C_Small") (at 96.52 130.81 0) (mirror y) (unit 1)
     (in_bom yes) (on_board yes) (fields_autoplaced)
-    (property "Reference" "C26" (id 0) (at 93.98 129.54 0)
+    (property "Reference" "C28" (id 0) (at 93.98 129.54 0)
       (effects (font (size 1.27 1.27)) (justify left))
     )
@@
   (symbol (lib_id "Device:R_Small") (at 149.86 92.71 0) (mirror x) (unit 1)
     (in_bom yes) (on_board yes)
-    (property "Reference" "R51" (id 0) (at 151.384 91.44 0)
+    (property "Reference" "R54" (id 0) (at 151.384 91.44 0)
       (effects (font (size 1.27 1.27)) (justify left))
     )
@@
   (symbol (lib_id "power:GND") (at 85.09 138.43 0) (mirror y) (unit 1)
     (in_bom yes) (on_board yes)
-    (property "Reference" "#PWR037" (id 0) (at 85.09 144.78 0)
-      (effects (font (size 1.27 1.27)) hide)
-    )
+    (property "Reference" "#PWR038" (id 0) (at 85.09 144.78 0)
+      (effects (font (size 1.27 1.27)) hide)
+    )
