File: psu5v.kicad_sch (KiCad schematic)
At the start: 26 parts, among them U16 AP64501SP-13

Commit message: leds
Parts:
- removed D3: LED Green, LED_SMD_LiteOn:LED_0603_1608Metric_green, symbol LED_SMD_LiteOn:LED Green
- C57: now left out of the parts list
- R66: value 1k -> 600R
Connections:
- net GND: no longer C57.2
- net +5V_OK: now reaches R66.2
- net at R63.1, U16.6 (COMP): no longer C57.1
- no-connect marks 2 -> 4
Other:
- note added: "< PSU On LED"
- note removed: "< PSU On"
Changed lines of the file:
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@@
   (junction (at 228.6 106.68) (diameter 1.016) (color 0 0 0 0)
   )
-  (junction (at 201.93 125.73) (diameter 1.016) (color 0 0 0 0)
-  )
   (junction (at 226.06 106.68) (diameter 0.9144) (color 0 0 0 0)
   )
@@
   (junction (at 191.77 106.68) (diameter 1.016) (color 0 0 0 0)
   )
-  (junction (at 201.93 147.32) (diameter 1.016) (color 0 0 0 0)
-  )
   (junction (at 121.92 123.19) (diameter 0.9144) (color 0 0 0 0)
   )
@@
   (junction (at 152.4 123.19) (diameter 0.9144) (color 0 0 0 0)
   )
+  (no_connect (at 201.93 134.62))
+  (no_connect (at 201.93 139.7))
   (no_connect (at 232.41 120.65))
   (no_connect (at 232.41 115.57))
@@
     (stroke (width 0) (type solid) (color 0 0 0 0))
   )
+  (wire (pts (xy 321.945 113.03) (xy 331.47 113.03))
+    (stroke (width 0) (type default) (color 0 0 0 0))
+  )
   (wire (pts (xy 248.92 116.84) (xy 259.08 116.84))
     (stroke (width 0) (type solid) (color 0 0 0 0))
@@
   )
   (wire (pts (xy 290.83 109.22) (xy 290.83 106.68))
-    (stroke (width 0) (type solid) (color 0 0 0 0))
-  )
-  (wire (pts (xy 201.93 125.73) (xy 201.93 134.62))
     (stroke (width 0) (type solid) (color 0 0 0 0))
   )
@@
     (stroke (width 0) (type default) (color 0 0 0 0))
   )
-  (wire (pts (xy 306.705 123.825) (xy 306.705 148.59))
-    (stroke (width 0) (type solid) (color 0 0 0 0))
-  )
   (wire (pts (xy 106.68 123.19) (xy 106.68 125.73))
     (stroke (width 0) (type solid) (color 0 0 0 0))
@@
     (stroke (width 0) (type solid) (color 0 0 0 0))
   )
-  (wire (pts (xy 201.93 125.73) (xy 213.36 125.73))
+  (wire (pts (xy 191.77 125.73) (xy 213.36 125.73))
     (stroke (width 0) (type solid) (color 0 0 0 0))
   )
@@
     (stroke (width 0) (type solid) (color 0 0 0 0))
   )
-  (wire (pts (xy 306.705 106.68) (xy 306.705 109.855))
+  (wire (pts (xy 306.705 106.68) (xy 306.705 113.03))
     (stroke (width 0) (type solid) (color 0 0 0 0))
   )
@@
     (stroke (width 0) (type solid) (color 0 0 0 0))
   )
-  (wire (pts (xy 194.31 147.32) (xy 201.93 147.32))
+  (wire (pts (xy 194.31 147.32) (xy 213.36 147.32))
     (stroke (width 0) (type solid) (color 0 0 0 0))
   )
@@
     (stroke (width 0) (type solid) (color 0 0 0 0))
   )
+  (wire (pts (xy 306.705 113.03) (xy 316.865 113.03))
+    (stroke (width 0) (type default) (color 0 0 0 0))
+  )
   (wire (pts (xy 259.08 106.68) (xy 259.08 109.22))
     (stroke (width 0) (type solid) (color 0 0 0 0))
@@
     (stroke (width 0) (type solid) (color 0 0 0 0))
   )
-  (wire (pts (xy 306.705 114.935) (xy 306.705 118.745))
-    (stroke (width 0) (type solid) (color 0 0 0 0))
-  )
   (wire (pts (xy 172.72 147.32) (xy 182.88 147.32))
     (stroke (width 0) (type solid) (color 0 0 0 0))
   )
-  (wire (pts (xy 191.77 125.73) (xy 201.93 125.73))
-    (stroke (width 0) (type solid) (color 0 0 0 0))
-  )
   (wire (pts (xy 191.77 106.68) (xy 191.77 120.65))
     (stroke (width 0) (type solid) (color 0 0 0 0))
@@
     (stroke (width 0) (type solid) (color 0 0 0 0))
   )
-  (wire (pts (xy 201.93 147.32) (xy 213.36 147.32))
-    (stroke (width 0) (type solid) (color 0 0 0 0))
-  )
   (wire (pts (xy 213.36 147.32) (xy 226.06 147.32))
     (stroke (width 0) (type solid) (color 0 0 0 0))
@@
     (stroke (width 0) (type solid) (color 0 0 0 0))
   )
+  (polyline (pts (xy 201.93 139.7) (xy 201.93 147.32))
+    (stroke (width 0) (type default) (color 0 0 0 0))
+  )
   (wire (pts (xy 279.4 106.68) (xy 279.4 109.22))
     (stroke (width 0) (type solid) (color 0 0 0 0))
   )
+  (polyline (pts (xy 201.93 125.73) (xy 201.93 134.62))
+    (stroke (width 0) (type default) (color 0 0 0 0))
+  )
   (wire (pts (xy 219.71 123.19) (xy 226.06 123.19))
     (stroke (width 0) (type solid) (color 0 0 0 0))
@@
     (stroke (width 0) (type solid) (color 0 0 0 0))
   )
-  (wire (pts (xy 201.93 139.7) (xy 201.93 147.32))
-    (stroke (width 0) (type solid) (color 0 0 0 0))
-  )
   (wire (pts (xy 248.92 114.3) (xy 248.92 116.84))
     (stroke (width 0) (type solid) (color 0 0 0 0))
@@
   (wire (pts (xy 213.36 143.51) (xy 213.36 147.32))
     (stroke (width 0) (type solid) (color 0 0 0 0))
+  )
+  (text "< PSU On LED" (at 344.805 113.665 0)
+    (effects (font (size 1.27 1.27)) (justify left bottom))
   )
   (text "+5V PSU @ 3A peak" (at 15.24 25.4 0)
@@
   (text "+5v @ 3A PSU ( 7.5v-28v Input )" (at 212.09 93.218 180)
     (effects (font (size 1.27 1.27)) (justify right bottom))
-  )
-  (text "< PSU On" (at 320.04 123.825 0)
-    (effects (font (size 1.27 1.27)) (justify left bottom))
   )
   (text "NB: Borrowed/Inspired by Raspberry Pi Foundation's CM4IO"
@@
     (effects (font (size 1.27 1.27)) (justify right))
   )
+  (hierarchical_label "+5V_OK" (shape output) (at 331.47 113.03 0)
+    (effects (font (size 1.27 1.27)) (justify left))
+  )
   (hierarchical_label "+5V_OUT" (shape output) (at 331.47 106.68 0)
     (effects (font (size 1.27 1.27)) (justify left))
@@
   (symbol (lib_id "power:GND") (at 152.4 148.59 0) (unit 1)
     (in_bom yes) (on_board yes)
-    (property "Reference" "#PWR049" (id 0) (at 152.4 154.94 0)
+    (property "Reference" "#PWR048" (id 0) (at 152.4 154.94 0)
       (effects (font (size 1.27 1.27)) hide)
     )
@@
     (pin "1")
   )
-  (symbol (lib_id "Device:R_Small") (at 306.705 112.395 0) (unit 1)
-    (in_bom yes) (on_board yes)
-    (property "Reference" "R66" (id 0) (at 309.88 111.125 0))
-    (property "Value" "1k" (id 1) (at 309.88 113.665 0))
-    (property "Footprint" "Resistor_SMD:R_0402_1005Metric" (id 2) (at 306.705 112.395 0)
-      (effects (font (size 1.27 1.27)) hide)
-    )
-    (property "Datasheet" "~" (id 3) (at 306.705 112.395 0)
-      (effects (font (size 1.27 1.27)) hide)
-    )
-    (pin "1")
-    (pin "2")
-  )
   (symbol (lib_id "power:GND") (at 290.83 148.59 0) (unit 1)
     (in_bom yes) (on_board yes)
-    (property "Reference" "#PWR053" (id 0) (at 290.83 154.94 0)
+    (property "Reference" "#PWR052" (id 0) (at 290.83 154.94 0)
       (effects (font (size 1.27 1.27)) hide)
     )
@@
   (symbol (lib_id "power:GND") (at 279.4 148.59 0) (unit 1)
     (in_bom yes) (on_board yes)
-    (property "Reference" "#PWR052" (id 0) (at 279.4 154.94 0)
+    (property "Reference" "#PWR051" (id 0) (at 279.4 154.94 0)
       (effects (font (size 1.27 1.27)) hide)
     )
@@
   (symbol (lib_id "power:GND") (at 226.06 148.59 0) (unit 1)
     (in_bom yes) (on_board yes)
-    (property "Reference" "#PWR050" (id 0) (at 226.06 154.94 0)
+    (property "Reference" "#PWR049" (id 0) (at 226.06 154.94 0)
       (effects (font (size 1.27 1.27)) hide)
     )
@@
     (pin "2")
   )
-  (symbol (lib_id "power:GND") (at 306.705 148.59 0) (unit 1)
-    (in_bom yes) (on_board yes)
-    (property "Reference" "#PWR054" (id 0) (at 306.705 154.94 0)
-      (effects (font (size 1.27 1.27)) hide)
-    )
-    (property "Value" "GND" (id 1) (at 306.705 152.4 0))
-    (property "Footprint" "" (id 2) (at 306.705 148.59 0)
-      (effects (font (size 1.27 1.27)) hide)
-    )
-    (property "Datasheet" "" (id 3) (at 306.705 148.59 0)
-      (effects (font (size 1.27 1.27)) hide)
-    )
-    (pin "1")
-  )
   (symbol (lib_id "Device:C_Small") (at 76.2 128.27 0) (unit 1)
     (in_bom yes) (on_board yes)
@@
   (symbol (lib_id "power:GND") (at 251.46 142.24 0) (unit 1)
     (in_bom yes) (on_board yes)
-    (property "Reference" "#PWR051" (id 0) (at 251.46 148.59 0)
+    (property "Reference" "#PWR050" (id 0) (at 251.46 148.59 0)
       (effects (font (size 1.27 1.27)) hide)
     )
@@
     (pin "2")
   )
+  (symbol (lib_id "Device:R_Small") (at 319.405 113.03 90) (unit 1)
+    (in_bom yes) (on_board yes)
+    (property "Reference" "R66" (id 0) (at 316.865 111.76 90)
+      (effects (font (size 1.27 1.27)) (justify left))
+    )
+    (property "Value" "600R" (id 1) (at 322.58 111.76 90)
+      (effects (font (size 1.27 1.27)) (justify right))
+    )
+    (property "Footprint" "Resistor_SMD:R_0402_1005Metric" (id 2) (at 319.405 113.03 0)
+      (effects (font (size 1.27 1.27)) hide)
+    )
+    (property "Datasheet" "~" (id 3) (at 319.405 113.03 0)
+      (effects (font (size 1.27 1.27)) hide)
+    )
+    (pin "1")
+    (pin "2")
+  )
   (symbol (lib_id "Device:C_Small") (at 201.93 137.16 0) (unit 1)
-    (in_bom yes) (on_board yes)
+    (in_bom no) (on_board no)
     (property "Reference" "C57" (id 0) (at 204.47 135.89 0)
       (effects (font (size 1.27 1.27)) (justify left))
@@
       (effects (font (size 1.27 1.27)) hide)
     )
-    (pin "1")
-    (pin "2")
-  )
-  (symbol (lib_id "LED_SMD_LiteOn:LED Green") (at 306.705 121.285 270) (unit 1)
-    (in_bom yes) (on_board yes)
-    (property "Reference" "D3" (id 0) (at 309.88 120.65 90))
-    (property "Value" "LED Green" (id 1) (at 313.69 122.555 90))
-    (property "Footprint" "LED_SMD_LiteOn:LED_0603_1608Metric_green" (id 2) (at 296.545 121.285 0)
-      (effects (font (size 1.27 1.27)) hide)
-    )
-    (property "Datasheet" "" (id 3) (at 306.705 121.285 90)
-      (effects (font (size 1.27 1.27)) hide)
-    )
-    (property "Manufacturer" "Lite-On" (id 4) (at 301.625 121.285 0)
-      (effects (font (size 1.27 1.27)) hide)
-    )
-    (property "MPN" "LTST-C193KGKT-5A" (id 5) (at 299.085 121.285 0)
-      (effects (font (size 1.27 1.27)) hide)
-    )

Commit message: led changes
Parts:
- R66: value 600R -> 580R
Changed lines of the file:
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@@
       (effects (font (size 1.27 1.27)) (justify left))
     )
-    (property "Value" "600R" (id 1) (at 322.58 111.76 90)
+    (property "Value" "580R" (id 1) (at 322.58 111.76 90)
       (effects (font (size 1.27 1.27)) (justify right))
     )
